File: pcb/androphage.kicad_pcb (KiCad board)
At the start: 2 copper layers, 83 parts, among them J1 VIK_OUT, J11 VIK_OUT_SENSOR, J12 Conn_01x04, J13 Conn_01x02, J2 Conn_01x04, J3 USB_C_Receptacle_USB2.0_16P, Q1 AO3401A, Q2 AO3401A, SW00 SW_Push_45deg, SW01 SW_Push_45deg, SW02 SW_Push_45deg, SW03 SW_Push_45deg, SW04 SW_Push_45deg, SW10 SW_Push_45deg, SW11 SW_Push_45deg, SW12 SW_Push_45deg, SW13 SW_Push_45deg, SW14 SW_Push_45deg, SW15 SW_Push_45deg, SW20 SW_Push_45deg, SW21 SW_Push_45deg, SW22 SW_Push_45deg, SW23 SW_Push_45deg, SW24 SW_Push_45deg, SW25 SW_Push_45deg, SW31 SW_Push_45deg, SW32 SW_Push_45deg, SW33 SW_Push_45deg, SW34 SW_Push_45deg, SW35 SW_Push_45deg, SW6 SW_Push, SW7 SW_SPST, U1 holyiot-18010-no-underside, U2 MCP73832-2-OT, U3 XC6220B331MR, U4 SRV05-4, U6 MCP23017_SO

Commit message: Start PCB layout.
Parts:
- U6: value MCP23017_SO -> MCP23017_SS; footprint Package_SO:SOIC-28W_7.5x17.9mm_P1.27mm -> Package_SO:SSOP-28_5.3x10.2mm_P0.65mm
- moved SW10 260.1 mm to (272.0, 65.5), turned to 90 degrees
- moved SW00 259.1 mm to (272.0, 48.5), turned to 90 degrees
- moved SW01 239.2 mm to (254.0, 40.0), turned to 90 degrees
- moved SW20 237.8 mm to (272.0, 82.5), turned to 90 degrees
- moved SW11 222.5 mm to (254.0, 57.0), turned to 90 degrees
- moved SW02 222.0 mm to (236.0, 31.5), turned to 90 degrees
- moved SW21 206.5 mm to (254.0, 74.0), turned to 90 degrees
- moved SW03 205.2 mm to (218.0, 40.0), turned to 90 degrees
- moved SW12 201.3 mm to (236.0, 48.5), turned to 90 degrees
- moved SW31 198.9 mm to (254.0, 91.0), turned to 90 degrees
- moved SW04 191.0 mm to (200.0, 40.0), turned to 90 degrees
- moved SW22 183.1 mm to (236.0, 65.5), turned to 90 degrees
- moved SW13 182.8 mm to (218.0, 57.0), turned to 90 degrees
- moved SW32 173.1 mm to (236.0, 82.5), turned to 90 degrees
- moved SW14 165.3 mm to (200.0, 57.0), turned to 90 degrees
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Routing:
- net /C4: track 0.00 -> 65.6 mm
- net Net-(D27-K): track 0.00 -> 14.1 mm
- net Net-(D6-K): track 0.00 -> 10.6 mm

Commit message: Update key switch footprint.
Parts:
- added R1: 10K, Resistor_SMD:R_0201_0603Metric_Pad0.64x0.40mm_HandSolder, F.Cu at (0.91, 0.38)
- SW00, SW01, SW02, SW03, SW04, SW10, SW11, SW12, SW13, SW14, SW15, SW20, SW21, SW22, SW23, SW24, SW25, SW31, SW32, SW33, SW34, SW35: footprint key-switches:SW_GLP_Kailh_Choc_V1V2_HotSwap_double -> key-switches:SW_Kailh_Choc_V1V2_HotSwap_PTH_Double
Connections:
- U6 pad 18: /GND -> Net-(U6-~{RESET})
Routing:
- net Net-(D6-K): track 10.6 -> 0.00 mm
- net /C4: track 65.6 -> 76.1 mm

Commit message: Restart PCB design.
Parts:
- removed D1: 1N5819WS, Diode_SMD:D_SOD-323
- removed D10, D11, D8, D9: SK6812MINI, LED_SMD:LED_SK6812MINI_PLCC4_3.5x3.5mm_P1.75mm
- removed D12, D13, D14, D15, D16, D17, D18, D19, D2, D20, D21, D22, D23, D24, D25, D26, D27, D28, D29, D3, D4, D5, D6, D7: 1N4148W, Diode_SMD:D_SOD-123
- removed F2: SMD0805-050-16V, Fuse:Fuse_0805_2012Metric
- removed FB2: ~, Inductor_SMD:L_0805_2012Metric
- removed J1: VIK_OUT, vik:vik-keyboard-connector-horizontal
- removed J11: VIK_OUT_SENSOR, vik:vik-keyboard-connector-horizontal
- removed J12: Conn_01x04, Connector_PinSocket_2.54mm:PinSocket_1x04_P2.54mm_Vertical
- removed J13: Conn_01x02, Connector_JST:JST_GH_SM02B-GHS-TB_1x02-1MP_P1.25mm_Horizontal
- removed J2: Conn_01x04, Connector_JST:JST_GH_SM04B-GHS-TB_1x04-1MP_P1.25mm_Horizontal
- removed J3: USB_C_Receptacle_USB2.0_16P, Connector_USB:USB_C_Receptacle_HRO_TYPE-C-31-M-12
- removed JP1: Charge_Boost, Jumper:SolderJumper-2_P1.3mm_Open_RoundedPad1.0x1.5mm
- removed Q1, Q2: AO3401A, Package_TO_SOT_SMD:SOT-23
- removed R1, R2, R3, R4, R5, R6, R7: 10K, Resistor_SMD:R_0201_0603Metric_Pad0.64x0.40mm_HandSolder
- removed R10: 100K, Resistor_SMD:R_0201_0603Metric_Pad0.64x0.40mm_HandSolder
- removed R11: 8K2, Resistor_SMD:R_0201_0603Metric_Pad0.64x0.40mm_HandSolder
- removed R12: 2K, Resistor_SMD:R_0201_0603Metric_Pad0.64x0.40mm_HandSolder
- removed R15: 820K, Resistor_SMD:R_0603_1608Metric
- removed R16, R17: 2M, Resistor_SMD:R_0603_1608Metric
- removed R8, R9: 5.1K, Resistor_SMD:R_0201_0603Metric_Pad0.64x0.40mm_HandSolder
- removed SW00, SW01, SW02, SW03, SW04, SW10, SW11, SW12, SW13, SW14, SW15, SW20, SW21, SW22, SW23, SW24, SW25, SW31, SW32, SW33, SW34, SW35: SW_Push_45deg, key-switches:SW_Kailh_Choc_V1V2_HotSwap_PTH_Double
- removed SW6: SW_Push, Button_Switch_SMD:SW_Push_1P1T_NO_E-Switch_TL3301NxxxxxG
- removed SW7: SW_SPST, library:AS11CH
- removed U1: holyiot-18010-no-underside, mcu:holyiot-18010-no-underside
- removed U2: MCP73832-2-OT, Package_TO_SOT_SMD:SOT-23-5
- removed U3: XC6220B331MR, Package_TO_SOT_SMD:SOT-23-5
- removed U4: SRV05-4, Package_TO_SOT_SMD:SOT-23-6
- removed U6: MCP23017_SS, Package_SO:SSOP-28_5.3x10.2mm_P0.65mm
- added D_LED_01: SK6812MINI, LED_SMD:LED_SK6812MINI_PLCC4_3.5x3.5mm_P1.75mm, F.Cu at (193.2, 93.9)
- added D_LED_02: SK6812MINI, LED_SMD:LED_SK6812MINI_PLCC4_3.5x3.5mm_P1.75mm, F.Cu at (193.2, 99.0)
- added D_LED_03: SK6812MINI, LED_SMD:LED_SK6812MINI_PLCC4_3.5x3.5mm_P1.75mm, F.Cu at (193.2, 104.1)
- added D_LED_04: SK6812MINI, LED_SMD:LED_SK6812MINI_PLCC4_3.5x3.5mm_P1.75mm, F.Cu at (193.2, 109.2)
- added D_POW_1: 1N5819WS, Diode_SMD:D_SOD-323, F.Cu at (197.6, 156.6)
- added F_USB_01: ~, Inductor_SMD:L_0805_2012Metric, F.Cu at (240.9, 164.2)
- added F_USB_02: SMD0805-050-16V, Fuse:Fuse_0805_2012Metric, F.Cu at (252.5, 174.5)
- added JP_CHG_01: Charge_Boost, Jumper:SolderJumper-2_P1.3mm_Open_RoundedPad1.0x1.5mm, F.Cu at (344.5, 168.8)
- added J_BAT_01: Conn_01x02, Connector_JST:JST_GH_SM02B-GHS-TB_1x02-1MP_P1.25mm_Horizontal, F.Cu at (354.8, 174.5)
- added J_OLED_01: Conn_01x04, Connector_JST:JST_GH_SM04B-GHS-TB_1x04-1MP_P1.25mm_Horizontal, F.Cu at (142.2, 103.8)
- added J_SWD_01: Conn_01x04, Connector_PinSocket_2.54mm:PinSocket_1x04_P2.54mm_Vertical, F.Cu at (207.5, 190.7)
- added J_USB_01: USB_C_Receptacle_USB2.0_16P, Connector_USB:USB_C_Receptacle_HRO_TYPE-C-31-M-12, F.Cu at (287.1, 164.9)
- added J_VIK_01: VIK_OUT, vik:vik-keyboard-connector-horizontal, F.Cu at (283.0, 233.8)
- added J_VIK_02: VIK_OUT_SENSOR, vik:vik-keyboard-connector-horizontal, F.Cu at (286.5, 208.8)
- added Q_EXT_01: AO3401A, Package_TO_SOT_SMD:SOT-23, F.Cu at (219.9, 159.1)
- added Q_POW_1: AO3401A, Package_TO_SOT_SMD:SOT-23, F.Cu at (193.0, 155.2)
- added REF**: MountingHole_2.2mm_M2, MountingHole:MountingHole_2.2mm_M2, F.Cu at (175.5, 217.3)
- added REF**: MountingHole_2.2mm_M2, MountingHole:MountingHole_2.2mm_M2, F.Cu at (269.8, 162.1)
- added REF**: MountingHole_2.2mm_M2, MountingHole:MountingHole_2.2mm_M2, F.Cu at (301.4, 249.2)
- added REF**: MountingHole_2.2mm_M2, MountingHole:MountingHole_2.2mm_M2, F.Cu at (301.4, 174.5)
- added REF**: MountingHole_2.2mm_M2, MountingHole:MountingHole_2.2mm_M2, F.Cu at (301.4, 205.8)
- added REF**: MountingHole_2.2mm_M2, MountingHole:MountingHole_2.2mm_M2, F.Cu at (281.1, 260.6)
- added REF**: MountingHole_2.2mm_M2, MountingHole:MountingHole_2.2mm_M2, F.Cu at (203.3, 144.8)
- added REF**: MountingHole_2.2mm_M2, MountingHole:MountingHole_2.2mm_M2, F.Cu at (165.0, 187.3)
- added R_CHG_01: 8K2, Resistor_SMD:R_0201_0603Metric_Pad0.64x0.40mm_HandSolder, F.Cu at (345.3, 174.9)
- added R_CHG_02: 2K, Resistor_SMD:R_0201_0603Metric_Pad0.64x0.40mm_HandSolder, F.Cu at (345.3, 176.6)
- added R_EXT_01: 2M, Resistor_SMD:R_0603_1608Metric, F.Cu at (220.9, 152.8)
- added R_MAT_01: 10K, Resistor_SMD:R_0201_0603Metric_Pad0.64x0.40mm_HandSolder, B.Cu at (123.5, 68.5)
- added R_MAT_02: 10K, Resistor_SMD:R_0201_0603Metric_Pad0.64x0.40mm_HandSolder, B.Cu at (118.5, 68.5)
- added R_MAT_11: 10K, Resistor_SMD:R_0201_0603Metric_Pad0.64x0.40mm_HandSolder, B.Cu at (123.5, 69.5)
- added R_MAT_12: 10K, Resistor_SMD:R_0201_0603Metric_Pad0.64x0.40mm_HandSolder, B.Cu at (118.5, 69.5)
- added R_MAT_21: 10K, Resistor_SMD:R_0201_0603Metric_Pad0.64x0.40mm_HandSolder, B.Cu at (123.5, 70.5)
- added R_MAT_22: 10K, Resistor_SMD:R_0201_0603Metric_Pad0.64x0.40mm_HandSolder, B.Cu at (118.5, 70.5)
- added R_MAT_31: 10K, Resistor_SMD:R_0201_0603Metric_Pad0.64x0.40mm_HandSolder, B.Cu at (118.4, 71.5)
- added R_MON_01: 820K, Resistor_SMD:R_0603_1608Metric, F.Cu at (334.4, 167.5)
- added R_MON_02: 2M, Resistor_SMD:R_0603_1608Metric, F.Cu at (334.4, 170.0)
- added R_POW_01: 100K, Resistor_SMD:R_0201_0603Metric_Pad0.64x0.40mm_HandSolder, F.Cu at (192.0, 162.0)
- added R_USB_01: 5.1K, Resistor_SMD:R_0201_0603Metric_Pad0.64x0.40mm_HandSolder, F.Cu at (265.8, 174.6)
- added R_USB_02: 5.1K, Resistor_SMD:R_0201_0603Metric_Pad0.64x0.40mm_HandSolder, F.Cu at (265.8, 176.3)
- added SW_BAT_01: SW_SPST, library:AS11CH, F.Cu at (288.5, 175.7)
- added SW_RST1: SW_Push, Button_Switch_SMD:SW_Push_1P1T_NO_E-Switch_TL3301NxxxxxG, F.Cu at (252.2, 82.5)
- added S_MAT_00: SW_Push_45deg, key-switches:SW_Kailh_Choc_V1V2_HotSwap_PTH_Double, F.Cu at (28.0, 40.5)
- added S_MAT_01: SW_Push_45deg, key-switches:SW_Kailh_Choc_V1V2_HotSwap_PTH_Double, F.Cu at (57.4, 30.5)
- added S_MAT_02: SW_Push_45deg, key-switches:SW_Kailh_Choc_V1V2_HotSwap_PTH_Double, F.Cu at (82.7, 31.9)
- added S_MAT_03: SW_Push_45deg, key-switches:SW_Kailh_Choc_V1V2_HotSwap_PTH_Double, F.Cu at (99.1, 40.6)
- added S_MAT_04: SW_Push_45deg, key-switches:SW_Kailh_Choc_V1V2_HotSwap_PTH_Double, F.Cu at (116.4, 45.3)
- added S_MAT_10: SW_Push_45deg, key-switches:SW_Kailh_Choc_V1V2_HotSwap_PTH_Double, F.Cu at (28.0, 57.5)
- added S_MAT_11: SW_Push_45deg, key-switches:SW_Kailh_Choc_V1V2_HotSwap_PTH_Double, F.Cu at (54.5, 47.2)
- added S_MAT_12: SW_Push_45deg, key-switches:SW_Kailh_Choc_V1V2_HotSwap_PTH_Double, F.Cu at (78.3, 48.3)
- added S_MAT_13: SW_Push_45deg, key-switches:SW_Kailh_Choc_V1V2_HotSwap_PTH_Double, F.Cu at (94.7, 57.0)
- added S_MAT_14: SW_Push_45deg, key-switches:SW_Kailh_Choc_V1V2_HotSwap_PTH_Double, F.Cu at (112.0, 61.7)
- added S_MAT_15: SW_Push_45deg, key-switches:SW_Kailh_Choc_V1V2_HotSwap_PTH_Double, F.Cu at (130.6, 92.3)
- added S_MAT_20: SW_Push_45deg, key-switches:SW_Kailh_Choc_V1V2_HotSwap_PTH_Double, F.Cu at (28.0, 74.5)
- added S_MAT_21: SW_Push_45deg, key-switches:SW_Kailh_Choc_V1V2_HotSwap_PTH_Double, F.Cu at (51.5, 64.0)
- added S_MAT_22: SW_Push_45deg, key-switches:SW_Kailh_Choc_V1V2_HotSwap_PTH_Double, F.Cu at (73.9, 64.7)
- added S_MAT_23: SW_Push_45deg, key-switches:SW_Kailh_Choc_V1V2_HotSwap_PTH_Double, F.Cu at (90.3, 73.4)
- added S_MAT_24: SW_Push_45deg, key-switches:SW_Kailh_Choc_V1V2_HotSwap_PTH_Double, F.Cu at (107.6, 78.1)
- added S_MAT_25: SW_Push_45deg, key-switches:SW_Kailh_Choc_V1V2_HotSwap_PTH_Double, F.Cu at (120.9, 106.2)
- added S_MAT_31: SW_Push_45deg, key-switches:SW_Kailh_Choc_V1V2_HotSwap_PTH_Double, F.Cu at (48.5, 80.7)
- added S_MAT_32: SW_Push_45deg, key-switches:SW_Kailh_Choc_V1V2_HotSwap_PTH_Double, F.Cu at (69.5, 81.1)
- added S_MAT_33: SW_Push_45deg, key-switches:SW_Kailh_Choc_V1V2_HotSwap_PTH_Double, F.Cu at (85.9, 89.9)
- added S_MAT_34: SW_Push_45deg, key-switches:SW_Kailh_Choc_V1V2_HotSwap_PTH_Double, F.Cu at (104.0, 96.6)
- added S_MAT_35: SW_Push_45deg, key-switches:SW_Kailh_Choc_V1V2_HotSwap_PTH_Double, F.Cu at (135.8, 118.7)
- added U_CHG_01: MCP73832-2-OT, Package_TO_SOT_SMD:SOT-23-5, F.Cu at (336.8, 177.0)
- added U_MAT_01: MCP23017_SS, Package_SO:SSOP-28_5.3x10.2mm_P0.65mm, F.Cu at (124.5, 72.5)
- added U_MCU_1: holyiot-18010-no-underside, mcu:holyiot-18010-no-underside, F.Cu at (263.5, 211.0)
- added U_POW_01: XC6220B331MR, Package_TO_SOT_SMD:SOT-23-5, F.Cu at (199.1, 149.4)
- added U_USB_01: SRV05-4, Package_TO_SOT_SMD:SOT-23-6, F.Cu at (242.2, 179.3)
Routing:
- net /R1: track 0.00 -> 188.9 mm
- net /R2: track 0.00 -> 180.8 mm, vias 0 -> 1
- net /R3: track 0.00 -> 169.7 mm
- net /R0: track 0.00 -> 169.5 mm
- net /C1: track 0.00 -> 162.6 mm, vias 0 -> 1
- net /C0: track 0.00 -> 161.8 mm, vias 0 -> 1
- net /C2: track 0.00 -> 132.6 mm, vias 0 -> 1
- net /C3: track 0.00 -> 124.2 mm, vias 0 -> 1
- net /C5: track 0.00 -> 79.0 mm, vias 0 -> 1
- net /C4: track 76.1 -> 102.5 mm, vias 0 -> 1
- net Net-(D27-K): track 14.1 -> 0.00 mm
- net Net-(U_MAT_01-A2): track 0.00 -> 4.98 mm, vias 0 -> 2
- net Net-(U_MAT_01-A1): track 0.00 -> 4.66 mm, vias 0 -> 2
- net Net-(U_MAT_01-A0): track 0.00 -> 4.37 mm, vias 0 -> 2
- net Net-(U_MAT_01-~{RESET}): track 0.00 -> 4.00 mm, vias 0 -> 1
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- added copper zone on B.Cu, net /GND
- added copper zone on F.Cu, net /GND
Other:
- board outline added: 290 x 254.1 mm
- board text added: "Bottom Plate"
- board text added: "Magnetic Connector"
- board text added: "Main PCB"
- board text added: "Switch Plate"
- board text added: "Trackball Sensor"

Commit message: Work on PCBs.
Parts:
- removed D_LED_01, D_LED_02, D_LED_03, D_LED_04: SK6812MINI, LED_SMD:LED_SK6812MINI_PLCC4_3.5x3.5mm_P1.75mm
- removed J_OLED_01: Conn_01x04, Connector_JST:JST_GH_SM04B-GHS-TB_1x04-1MP_P1.25mm_Horizontal
- removed the REF** at (175.5, 217.3)
- removed the REF** at (269.8, 162.1)
- removed the REF** at (301.4, 249.2)
- removed the REF** at (301.4, 174.5)
- removed the REF** at (301.4, 205.8)
- removed the REF** at (281.1, 260.6)
- removed the REF** at (203.3, 144.8)
- removed the REF** at (165.0, 187.3)
- added J_VIK_03: VIK_OUT_DISP, vik:vik-keyboard-connector-horizontal, F.Cu at (62.6, 176.5)
- added REF**: PinSocket_1x01_P2.54mm_Vertical, Connector_PinSocket_2.54mm:PinSocket_1x01_P2.54mm_Vertical, F.Cu at (325.0, 26.5)
- added REF**: PinSocket_1x01_P2.54mm_Vertical, Connector_PinSocket_2.54mm:PinSocket_1x01_P2.54mm_Vertical, F.Cu at (340.0, 26.5)
- added REF**: PinSocket_1x04_P2.54mm_Vertical, Connector_PinSocket_2.54mm:PinSocket_1x04_P2.54mm_Vertical, F.Cu at (336.5, 39.0)
- J_VIK_01: value VIK_OUT -> VIK_OUT_INTC
- J_VIK_02: value VIK_OUT_SENSOR -> VIK_OUT_SENS
- moved SW_RST1 199.5 mm to (117.5, 229.5)
- moved U_USB_01 170.0 mm to (332.6, 35.4)
- moved F_USB_02 163.7 mm to (339.0, 35.5), turned to -90 degrees
- moved R_USB_01 156.2 mm to (335.0, 34.5), turned to -90 degrees
- moved R_USB_02 155.3 mm to (329.0, 34.5), turned to -90 degrees
- moved FB_USB_01 154.3 mm to (326.0, 35.4), turned to -90 degrees
- moved U_MCU_1 148.2 mm to (116.5, 192.0)
- moved JP_CHG_01 148.1 mm to (196.5, 165.6)
- moved R_MON_01 148.1 mm to (186.4, 164.3)
- moved R_MON_02 148.1 mm to (186.4, 166.8)
- moved D_POW_1 148.1 mm to (49.5, 153.4)
- moved J_BAT_01 148.1 mm to (206.8, 171.4)
- moved J_VIK_01 148.1 mm to (135.0, 230.6)
- moved J_VIK_02 148.1 mm to (138.5, 205.6)
- moved Q_EXT_01 148.1 mm to (71.9, 155.9)
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- renumbered F_USB_01 to FB_USB_01
Connections:
- J_SWD_01 pad 2: /GND -> /SWC
- J_SWD_01 pad 3: /SWD -> /GND
- J_SWD_01 pad 4: /SWC -> /SWD
- SW_RST1 pad 1: Net-(U_MCU_1-P0.19) -> Net-(U_MCU_1-Reset/P0.18)
- U_MCU_1 pad 35: /INT_PMW1 -> /CS_PMW2
- U_MCU_1 pad 36: /GP12 -> /CS_DIS1
- U_MCU_1 pad 39: /CS_PMW2 -> /INT_PMW1
- U_MCU_1 pad 41: /GP22 -> /GP31
- U_MCU_1 pad 48: unconnected-(U_MCU_1-Reset/P0.18-Pad48) -> Net-(U_MCU_1-Reset/P0.18)
- U_MCU_1 pad 49: Net-(U_MCU_1-P0.19) -> /GP32
- U_MCU_1 pad 50: unconnected-(U_MCU_1-P0.21-Pad50) -> /GP22
- U_MCU_1 pad 51: unconnected-(U_MCU_1-P0.23-Pad51) -> /GP12
- U_MCU_1 pad 6: unconnected-(U_MCU_1-[L]_A1_P0.03-Pad6) -> /RGB_DO3
Routing:
- net /GNDPWR: track 0.00 -> 21.6 mm
- net /VBUS: track 0.00 -> 19.9 mm
- net /VDD: track 0.00 -> 17.1 mm, vias 0 -> 1
- net /GND: track 0.00 -> 15.8 mm, vias 1 -> 9
- net /D-: track 0.00 -> 11.5 mm
- net /D+: track 0.00 -> 10.4 mm
- net /R3: track 169.7 -> 160.0 mm
- net /5V: track 0.00 -> 3.60 mm
- net Net-(J_USB_01-CC2): track 0.00 -> 3.02 mm
- net Net-(J_USB_01-CC1): track 0.00 -> 2.57 mm
- net /C4: track 102.5 -> 101.7 mm
Other:
- board size 290 x 254.1 mm -> 325.8 x 250.9 mm
- board text added: "Bottom Plates"
- board text added: "USB Daughterboard"
- board text removed: "Bottom Plate"
- board text removed: "Magnetic Connector"
- board text removed: "Trackball Sensor"

Commit message: Relocate USB connector to switch PCB.
Parts:
- added FB_USB_01: ~, Inductor_SMD:L_0805_2012Metric, B.Cu at (70.5, 16.0)
- added F_USB_02: SMD0805-050-16V, Fuse:Fuse_0805_2012Metric, B.Cu at (70.5, 24.2)
- added J_USB_01: USB_C_Receptacle_USB2.0_16P, Connector_USB:USB_C_Receptacle_HRO_TYPE-C-31-M-12, B.Cu at (63.0, 16.5)
- added R_USB_01: 5.1K, Resistor_SMD:R_0201_0603Metric_Pad0.64x0.40mm_HandSolder, B.Cu at (70.0, 22.5)
- added R_USB_02: 5.1K, Resistor_SMD:R_0201_0603Metric_Pad0.64x0.40mm_HandSolder, B.Cu at (70.0, 18.2)
- added U_USB_01: SRV05-4, Package_TO_SOT_SMD:SOT-23-6, B.Cu at (71.1, 20.3)
Routing:
- net /VBUS: track 19.9 -> 48.0 mm
- net /GNDPWR: track 21.6 -> 40.9 mm
- net /D-: track 11.5 -> 29.3 mm
- net /D+: track 10.4 -> 27.2 mm
- net Net-(J_USB_01-CC1): track 2.57 -> 12.1 mm
- net Net-(J_USB_01-CC2): track 3.02 -> 10.9 mm
- net /GND: track 15.8 -> 19.2 mm, vias 9 -> 13

Commit message: Work on PCBs.
Parts:
- removed D_POW_1: 1N5819WS, Diode_SMD:D_SOD-323
- removed the FB_USB_01 at (70.5, 16.0)
- removed the F_USB_02 at (70.5, 24.2)
- removed the J_USB_01 at (63.0, 16.5)
- removed J_VIK_01: VIK_OUT_INTC, vik:vik-keyboard-connector-horizontal
- removed J_VIK_02: VIK_OUT_SENS, vik:vik-keyboard-connector-horizontal
- removed J_VIK_03: VIK_OUT_DISP, vik:vik-keyboard-connector-horizontal
- removed Q_POW_1: AO3401A, Package_TO_SOT_SMD:SOT-23
- removed REF** (x2): PinSocket_1x01_P2.54mm_Vertical, Connector_PinSocket_2.54mm:PinSocket_1x01_P2.54mm_Vertical
- removed REF**: PinSocket_1x04_P2.54mm_Vertical, Connector_PinSocket_2.54mm:PinSocket_1x04_P2.54mm_Vertical
- removed the R_USB_01 at (70.0, 22.5)
- removed the R_USB_02 at (70.0, 18.2)
- removed SW_RST1: SW_Push, Button_Switch_SMD:SW_Push_1P1T_NO_E-Switch_TL3301NxxxxxG
- removed U_MCU_1: holyiot-18010-no-underside, mcu:holyiot-18010-no-underside
- removed the U_USB_01 at (71.1, 20.3)
- added D_POW_01: 1N5819WS, Diode_SMD:D_SOD-323, F.Cu at (127.0, 46.5)
- added J_VIK_IN_INTC_01: vik-module-connector, vik:vik-module-connector-horizontal, F.Cu at (186.5, 170.8)
- added J_VIK_IN_SW_01: vik-module-connector, vik:vik-module-connector-horizontal, F.Cu at (141.8, 103.2)
- added J_VIK_OUT_DISP_01: VIK_OUT_DISP, vik:vik-keyboard-connector-horizontal, F.Cu at (128.0, 202.0)
- added J_VIK_OUT_DISP_02: VIK_OUT_DISP, vik:vik-keyboard-connector-horizontal, F.Cu at (198.0, 170.8)
- added J_VIK_OUT_INTC_01: VIK_OUT_INTC, vik:vik-keyboard-connector-horizontal, F.Cu at (129.4, 190.5)
- added J_VIK_OUT_SENS_01: VIK_OUT_SENS, vik:vik-keyboard-connector-horizontal, F.Cu at (129.4, 213.5)
- added J_VIK_OUT_SENS_02: VIK_OUT_SENS, vik:vik-keyboard-connector-horizontal, F.Cu at (198.0, 181.8)
- added J_VIK_OUT_SW_01: VIK_OUT_SW, vik:vik-keyboard-connector-horizontal, F.Cu at (128.0, 225.0)
- added J_VIK_OUT_SW_02: VIK_OUT_SW, vik:vik-keyboard-connector-horizontal, F.Cu at (198.0, 192.8)
- added Q_POW_01: AO3401A, Package_TO_SOT_SMD:SOT-23, F.Cu at (127.0, 49.5)
- added SW_RST_01: SW_Push, Button_Switch_SMD:SW_Push_1P1T_NO_E-Switch_TL3301NxxxxxG, F.Cu at (277.5, 80.0)
- added U_MCU_01: holyiot-18010-no-underside, mcu:holyiot-18010-no-underside, F.Cu at (142.8, 169.2)
- FB_USB_01, SW_BAT_01: moved to B.Cu
- J_SWD_01: footprint Connector_PinSocket_2.54mm:PinSocket_1x04_P2.54mm_Vertical -> Connector_PinHeader_2.54mm:PinHeader_1x04_P2.54mm_Vertical_SMD_Pin1Left
- moved J_BAT_01 226.7 mm to (32.0, 27.0), turned to -90 degrees
- moved F_USB_02 208.0 mm to (131.0, 37.0), turned to 180 degrees
- moved R_USB_01 204.0 mm to (131.0, 34.5), turned to 180 degrees
- moved U_USB_01 202.1 mm to (130.5, 40.0), turned to 180 degrees
- moved R_USB_02 197.9 mm to (131.1, 35.5), turned to 180 degrees
- moved J_USB_01 194.7 mm to (138.0, 36.0)
- moved FB_USB_01 181.0 mm to (145.0, 39.0), turned to 0 degrees
- moved SW_BAT_01 178.0 mm to (201.5, 22.4)
- moved R_POW_01 142.5 mm to (129.0, 44.5)
- moved U_POW_01 116.2 mm to (127.0, 58.4), turned to -90 degrees
- moved U_CHG_01 62.8 mm to (250.0, 160.0)
- moved R_MON_02 59.8 mm to (245.0, 155.0)
- moved Q_EXT_01 58.5 mm to (129.5, 166.0), turned to 180 degrees
- moved R_EXT_01 54.8 mm to (125.5, 165.0), turned to 180 degrees
- moved R_MON_01 48.7 mm to (234.2, 155.0)
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Connections:
- net /BATT_MON renamed /Power_Board/BATT_MON
- net /C0 renamed /Switch_Board/C0
- net /C1 renamed /Switch_Board/C1
- net /C2 renamed /Switch_Board/C2
- net /C3 renamed /Switch_Board/C3
- net /C4 renamed /Switch_Board/C4
- net /C5 renamed /Switch_Board/C5
- net /D+ renamed /Switch_Board/D+
- net /D- renamed /Switch_Board/D-
- net /GNDPWR renamed /Switch_Board/GNDPWR
- net /R0 renamed /Switch_Board/R0
- net /R1 renamed /Switch_Board/R1
- net /R2 renamed /Switch_Board/R2
- net /R3 renamed /Switch_Board/R3
- net /VBUS renamed /Switch_Board/VBUS
- net /VEXT_EN renamed /Control_Board/VEXT_EN
- FB_USB_01 pad 2: /GND -> /Switch_Board/GND
- F_USB_02 pad 2: /5V -> /Switch_Board/5V
- J_BAT_01 pad 2: /GND -> /Switch_Board/GND
- J_BAT_01 pad MP: (no net) -> /Switch_Board/GND
- J_SWD_01 pad 1: /VDD -> /Control_Board/VDD
- J_SWD_01 pad 2: /SWC -> /Control_Board/SWC
- J_SWD_01 pad 3: /GND -> /Control_Board/GND
- J_SWD_01 pad 4: /SWD -> /Control_Board/SWD
- J_USB_01 pad A1: /GND -> /Switch_Board/GND
- J_USB_01 pad A12: /GND -> /Switch_Board/GND
- J_USB_01 pad B1: /GND -> /Switch_Board/GND
- J_USB_01 pad B12: /GND -> /Switch_Board/GND
- Q_EXT_01 pad 2: /VDD -> /Control_Board/VDD
- Q_EXT_01 pad 3: /VEXT -> /Control_Board/VEXT
- R_CHG_02 pad 2: /GND -> /Power_Board/GND
- R_EXT_01 pad 2: /GND -> /Control_Board/GND
- R_MAT_01 pad 2: /GND -> /Switch_Board/GND
- R_MAT_02 pad 1: /VDD -> /Switch_Board/VDD
- R_MAT_11 pad 2: /GND -> /Switch_Board/GND
- R_MAT_12 pad 1: /VDD -> /Switch_Board/VDD
- R_MAT_21 pad 2: /GND -> /Switch_Board/GND
- R_MAT_22 pad 1: /VDD -> /Switch_Board/VDD
- R_MAT_31 pad 1: /VDD -> /Switch_Board/VDD
- R_MON_01 pad 1: /VBAT -> /Power_Board/VBAT
- R_MON_02 pad 2: /GND -> /Power_Board/GND
- R_POW_01 pad 1: /5V -> /Switch_Board/5V
- R_POW_01 pad 2: /GND -> /Switch_Board/GND
- R_USB_01 pad 2: /GND -> /Switch_Board/GND
- R_USB_02 pad 2: /GND -> /Switch_Board/GND
- SW_BAT_01 pad 1: /VBAT -> /Switch_Board/VBAT
- SW_BAT_01 pad MH1: (no net) -> /Switch_Board/GND
- SW_BAT_01 pad MH2: (no net) -> /Switch_Board/GND
- U_CHG_01 pad 1: /CHG_STAT -> /Power_Board/CHG_STAT
- U_CHG_01 pad 2: /GND -> /Power_Board/GND
- U_CHG_01 pad 3: /VBAT -> /Power_Board/VBAT
- U_CHG_01 pad 4: /5V -> /Power_Board/5V
- U_MAT_01 pad 10: /GND -> /Switch_Board/GND
- U_MAT_01 pad 12: /SDA -> /Switch_Board/SDA
- U_MAT_01 pad 13: /SCL -> /Switch_Board/SCL
- U_MAT_01 pad 9: /VDD -> /Switch_Board/VDD
- U_POW_01 pad 2: /GND -> /Switch_Board/GND
- U_POW_01 pad 5: /VDD -> /Switch_Board/VDD
- U_USB_01 pad 2: /GND -> /Switch_Board/GND
Routing:
- net /Control_Board/VDD: track 0.00 -> 130.5 mm
- net /Switch_Board/VBAT: track 0.00 -> 98.3 mm
- net /Switch_Board/VDD: track 0.00 -> 61.9 mm, vias 0 -> 1
- net /Switch_Board/D+: track 27.2 -> 85.9 mm, vias 0 -> 2
- net /Control_Board/SDA: track 0.00 -> 56.0 mm
- net /Control_Board/SCL: track 0.00 -> 54.6 mm
- net /Switch_Board/GND: track 0.00 -> 54.2 mm, vias 0 -> 8
- net /Switch_Board/D-: track 29.3 -> 83.3 mm, vias 0 -> 2
- net /Control_Board/VEXT: track 0.00 -> 52.5 mm
- net /Switch_Board/RST: track 0.00 -> 51.3 mm
- net /Control_Board/MOSI: track 0.00 -> 50.3 mm
- net /Control_Board/MISO: track 0.00 -> 47.4 mm
- net /Control_Board/SCLK: track 0.00 -> 44.2 mm
- net /Power_Board/SCLK: track 0.00 -> 42.9 mm
- net /Switch_Board/SCL: track 0.00 -> 41.9 mm, vias 0 -> 2
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- added copper zone on B.Cu, net /Control_Board/GND
- added copper zone on F.Cu, net /Control_Board/GND
- added copper zone on B.Cu, net /Power_Board/GND
- added copper zone on F.Cu, net /Power_Board/GND
- added copper zone on B.Cu, net /Switch_Board/GND
- added copper zone on F.Cu, net /Switch_Board/GND
- removed copper zone on B.Cu, net /GND
- removed copper zone on F.Cu, net /GND
Other:
- board size 325.8 x 250.9 mm -> 289.9 x 251 mm
- board text removed: "USB Daughterboard"
