File: pcb/androphage.kicad_pcb (KiCad board)
At the start: 2 copper layers, 289.9 x 251 mm, 62 parts

Commit message: Work on PCBs.
Parts:
- removed J_VIK_OUT_DISP_02: VIK_OUT_DISP, vik:vik-keyboard-connector-horizontal
- added H1: MountingHole_Pad, MountingHole:MountingHole_2.2mm_M2_Pad, F.Cu at (55.4, 141.9)
- added H10: MountingHole_Pad, MountingHole:MountingHole_2.2mm_M2_Pad, F.Cu at (165.0, 201.7)
- added H11: MountingHole_Pad, MountingHole:MountingHole_2.2mm_M2_Pad, F.Cu at (256.8, 221.5)
- added H12: MountingHole_Pad, MountingHole:MountingHole_2.2mm_M2_Pad, F.Cu at (184.9, 257.6)
- added H2: MountingHole_Pad, MountingHole:MountingHole_2.2mm_M2_Pad, F.Cu at (122.0, 159.2)
- added H3: MountingHole_Pad, MountingHole:MountingHole_2.2mm_M2_Pad, F.Cu at (17.2, 184.4)
- added H4: MountingHole_Pad, MountingHole:MountingHole_2.2mm_M2_Pad, F.Cu at (153.3, 201.9)
- added H5: MountingHole_Pad, MountingHole:MountingHole_2.2mm_M2_Pad, F.Cu at (61.5, 221.7)
- added H6: MountingHole_Pad, MountingHole:MountingHole_2.2mm_M2_Pad, F.Cu at (133.4, 257.8)
- added H7: MountingHole_Pad, MountingHole:MountingHole_2.2mm_M2_Pad, F.Cu at (262.9, 141.7)
- added H8: MountingHole_Pad, MountingHole:MountingHole_2.2mm_M2_Pad, F.Cu at (196.3, 159.0)
- added H9: MountingHole_Pad, MountingHole:MountingHole_2.2mm_M2_Pad, F.Cu at (301.1, 184.2)
- added J1: Conn_01x04, Connector_PinHeader_2.54mm:PinHeader_1x04_P2.54mm_Vertical, F.Cu at (40.4, 43.7)
- added J2: Conn_01x04, Connector_PinHeader_2.54mm:PinHeader_1x04_P2.54mm_Vertical, F.Cu at (196.5, 44.0)
- moved U_CHG_01 96.7 mm to (189.0, 235.0), turned to 180 degrees
- moved R_MON_02 93.3 mm to (189.5, 230.0)
- moved R_MON_01 88.6 mm to (189.5, 231.5), turned to 180 degrees
- moved R_CHG_01 85.8 mm to (185.0, 238.0), turned to 180 degrees
- moved R_CHG_02 85.2 mm to (185.0, 239.0)
- moved JP_CHG_01 84.0 mm to (184.9, 236.0), turned to 180 degrees
- moved Q_EXT_01 78.5 mm to (53.1, 148.1)
- moved R_EXT_01 78.5 mm to (49.1, 147.1)
- moved U_MCU_01 75.8 mm to (69.0, 151.5)
- moved J_SWD_01 75.0 mm to (81.5, 151.5), turned to 180 degrees
- moved J_VIK_IN_INTC_01 59.1 mm to (178.3, 229.3), turned to 180 degrees
- moved J_VIK_OUT_SENS_01 45.4 mm to (140.0, 169.3), turned to 0 degrees
- moved J_VIK_OUT_INTC_01 40.2 mm to (140.0, 229.3), turned to 0 degrees
- moved J_VIK_OUT_SW_02 25.7 mm to (178.3, 209.3)
- moved J_VIK_OUT_SENS_02 23.3 mm to (178.3, 169.3)
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Connections:
- net /Switch_Board/GNDPWR renamed /Switch_Board/SH
- net /Switch_Board/VBUS renamed /Switch_Board/VUSB
- J_BAT_01 pad 1: Net-(J_BAT_01-Pin_1) -> /Switch_Board/GND
- J_BAT_01 pad 2: /Switch_Board/GND -> Net-(J1-Pin_1)
- J_BAT_01 pad MP: /Switch_Board/GND -> (no net)
- J_VIK_IN_INTC_01 pad 13: /Power_Board/GND -> (no net)
- J_VIK_IN_INTC_01 pad 14: /Power_Board/GND -> (no net)
- J_VIK_IN_INTC_01 pad 4: /Power_Board/GP22 -> /Power_Board/BATT_MON
- J_VIK_IN_INTC_01 pad 7: /Power_Board/VEXT -> /Power_Board/5V
- J_VIK_IN_INTC_01 pad 8: /Power_Board/RGB_DO2 -> /Power_Board/VEXT
- J_VIK_IN_SW_01 pad 1: /Switch_Board/VDD -> /Switch_Board/SCLK
- J_VIK_IN_SW_01 pad 10: /Switch_Board/RST -> /Switch_Board/SDA
- J_VIK_IN_SW_01 pad 11: /Switch_Board/MISO -> /Switch_Board/GND
- J_VIK_IN_SW_01 pad 12: /Switch_Board/SCLK -> /Switch_Board/VDD
- J_VIK_IN_SW_01 pad 13: /Switch_Board/GND -> (no net)
- J_VIK_IN_SW_01 pad 14: /Switch_Board/GND -> (no net)
- J_VIK_IN_SW_01 pad 2: /Switch_Board/GND -> /Switch_Board/MISO
- J_VIK_IN_SW_01 pad 3: /Switch_Board/SDA -> /Switch_Board/RST
- J_VIK_IN_SW_01 pad 4: /Switch_Board/SCL -> /Switch_Board/D+
- J_VIK_IN_SW_01 pad 5: /Switch_Board/RGB_DO1 -> /Switch_Board/MOSI
- J_VIK_IN_SW_01 pad 6: /Switch_Board/VEXT -> /Switch_Board/D-
- J_VIK_IN_SW_01 pad 7: /Switch_Board/D- -> /Switch_Board/5V
- J_VIK_IN_SW_01 pad 8: /Switch_Board/MOSI -> /Switch_Board/VEXT
- J_VIK_IN_SW_01 pad 9: /Switch_Board/D+ -> /Switch_Board/SCL
- J_VIK_OUT_DISP_01 pad 13: /Control_Board/GND -> (no net)
- J_VIK_OUT_DISP_01 pad 14: /Control_Board/GND -> (no net)
- J_VIK_OUT_DISP_01 pad 5: /Control_Board/RGB_DO1 -> /Control_Board/VEXT
- J_VIK_OUT_DISP_01 pad 6: /Control_Board/VEXT -> /Control_Board/5V
- J_VIK_OUT_INTC_01 pad 13: /Control_Board/GND -> (no net)
- J_VIK_OUT_INTC_01 pad 14: /Control_Board/GND -> (no net)
- J_VIK_OUT_INTC_01 pad 5: /Control_Board/RGB_DO2 -> /Control_Board/VEXT
- J_VIK_OUT_INTC_01 pad 6: /Control_Board/VEXT -> /Control_Board/5V
- J_VIK_OUT_SENS_01 pad 13: /Control_Board/GND -> (no net)
- J_VIK_OUT_SENS_01 pad 14: /Control_Board/GND -> (no net)
- J_VIK_OUT_SENS_01 pad 5: /Control_Board/RGB_DO1 -> /Control_Board/VEXT
- J_VIK_OUT_SENS_01 pad 6: /Control_Board/VEXT -> /Control_Board/5V
- J_VIK_OUT_SENS_02 pad 13: /Power_Board/GND -> (no net)
- J_VIK_OUT_SENS_02 pad 14: /Power_Board/GND -> (no net)
- J_VIK_OUT_SENS_02 pad 5: /Power_Board/RGB_DO2 -> /Power_Board/VEXT
- J_VIK_OUT_SENS_02 pad 6: /Power_Board/VEXT -> /Power_Board/5V
- J_VIK_OUT_SENS_02 pad 9: /Power_Board/GP12 -> unconnected-(J_VIK_OUT_SENS_02-GP_AD2-Pad9)
- J_VIK_OUT_SW_01 pad 13: /Control_Board/GND -> (no net)
- J_VIK_OUT_SW_01 pad 14: /Control_Board/GND -> (no net)
- J_VIK_OUT_SW_01 pad 5: /Control_Board/RGB_DO1 -> /Control_Board/VEXT
- J_VIK_OUT_SW_01 pad 6: /Control_Board/VEXT -> /Control_Board/5V
- J_VIK_OUT_SW_02 pad 10: /Power_Board/CS_SW2 -> unconnected-(J_VIK_OUT_SW_02-SPI_CS-Pad10)
- J_VIK_OUT_SW_02 pad 13: /Power_Board/GND -> (no net)
- J_VIK_OUT_SW_02 pad 14: /Power_Board/GND -> (no net)
- J_VIK_OUT_SW_02 pad 5: /Power_Board/RGB_DO2 -> /Power_Board/VEXT
- J_VIK_OUT_SW_02 pad 6: /Power_Board/VEXT -> /Power_Board/5V
- J_VIK_OUT_SW_02 pad 7: /Power_Board/D- -> unconnected-(J_VIK_OUT_SW_02-GP_AD1-Pad7)
- J_VIK_OUT_SW_02 pad 9: /Power_Board/D+ -> unconnected-(J_VIK_OUT_SW_02-GP_AD2-Pad9)
- SW_BAT_01 pad 1: /Switch_Board/VBAT -> Net-(J2-Pin_1)
- SW_BAT_01 pad 2: Net-(J_BAT_01-Pin_1) -> Net-(J2-Pin_2)
- SW_BAT_01 pad MH1: /Switch_Board/GND -> (no net)
- SW_BAT_01 pad MH2: /Switch_Board/GND -> (no net)
- SW_RST_01 pad 1: /Switch_Board/RST -> /Switch_Board/PLATE_GND
- SW_RST_01 pad 2: /Switch_Board/GND -> Net-(J2-Pin_4)
- U_MCU_01 pad 4: /Control_Board/RGB_DO1 -> unconnected-(U_MCU_01-[L]_P1.13-Pad4)
- U_MCU_01 pad 5: /Control_Board/RGB_DO2 -> unconnected-(U_MCU_01-[L]_P1.15-Pad5)
- U_MCU_01 pad 6: /Control_Board/RGB_DO3 -> unconnected-(U_MCU_01-[L]_A1_P0.03-Pad6)
Routing:
- net /Control_Board/5V: track 0.00 -> 178.9 mm
- net Net-(J2-Pin_4): track 0.00 -> 162.5 mm
- net /Switch_Board/RST: track 51.3 -> 207.6 mm, vias 0 -> 1
- net /Control_Board/INT_PMW2: track 0.00 -> 136.4 mm, vias 0 -> 2
- net /Control_Board/SCLK: track 44.2 -> 176.1 mm
- net /Control_Board/MISO: track 47.4 -> 173.8 mm
- net /Control_Board/GP22: track 0.00 -> 125.3 mm, vias 0 -> 2
- net /Control_Board/CS_PMW2: track 0.00 -> 120.5 mm, vias 0 -> 2
- net /Control_Board/GP12: track 0.00 -> 114.5 mm, vias 0 -> 2
- net /Control_Board/D-: track 0.00 -> 102.3 mm, vias 0 -> 2
- net /Control_Board/GP31: track 0.00 -> 100.6 mm, vias 0 -> 2
- net /Control_Board/D+: track 0.00 -> 100.5 mm, vias 0 -> 2
- net /Control_Board/GP32: track 0.00 -> 99.7 mm, vias 0 -> 2
- net /Control_Board/GND: track 0.00 -> 97.2 mm, vias 0 -> 4
- net /Control_Board/CS_DIS1: track 0.00 -> 96.4 mm, vias 0 -> 2
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- added copper zone on B.Cu, net /Switch_Board/PLATE_GND
- added copper zone on F.Cu, net /Switch_Board/PLATE_GND
Other:
- board size 289.9 x 251 mm -> 289.7 x 251.2 mm
