File: pcb/androphage.kicad_pcb (KiCad board)
At the start: 2 copper layers, 289.7 x 251.2 mm, 75 parts, among them J1 Conn_01x04, J2 Conn_01x04

Commit message: Split PCBs into separate projects.
Parts:
- added REF**: MouseBite-Slot_2.0x2.0mm_inset_D0.5mm_P0.85mm_5h, Panelization:MouseBite-Slot_2.0x2.0mm_inset_D0.5mm_P0.85mm_5h, F.Cu at (158.0, 171.0)
- added REF**: MouseBite-Slot_2.0x2.0mm_inset_D0.5mm_P0.85mm_5h, Panelization:MouseBite-Slot_2.0x2.0mm_inset_D0.5mm_P0.85mm_5h, F.Cu at (158.0, 197.0)
- added REF**: MouseBite-Slot_2.0x2.0mm_inset_D0.5mm_P0.85mm_5h, Panelization:MouseBite-Slot_2.0x2.0mm_inset_D0.5mm_P0.85mm_5h, F.Cu at (158.0, 131.1)
- added REF**: MouseBite-Slot_2.0x2.0mm_inset_D0.5mm_P0.85mm_5h, Panelization:MouseBite-Slot_2.0x2.0mm_inset_D0.5mm_P0.85mm_5h, F.Cu at (158.0, 223.0)
- added REF**: MouseBite-Slot_2.0x2.0mm_inset_D0.5mm_P0.85mm_5h, Panelization:MouseBite-Slot_2.0x2.0mm_inset_D0.5mm_P0.85mm_5h, F.Cu at (158.0, 249.0)
- added REF**: MouseBite-Slot_2.0x2.0mm_inset_D0.5mm_P0.85mm_5h, Panelization:MouseBite-Slot_2.0x2.0mm_inset_D0.5mm_P0.85mm_5h, F.Cu at (158.0, 113.1)
- added REF**: MouseBite-Slot_2.0x2.0mm_inset_D0.5mm_P0.85mm_5h, Panelization:MouseBite-Slot_2.0x2.0mm_inset_D0.5mm_P0.85mm_5h, F.Cu at (158.0, 151.1)
- J2, SW_RST_01: moved to B.Cu
- SW_BAT_01: moved to F.Cu
- moved SW_RST_01 95.6 mm to (184.6, 102.4), turned to -65 degrees
- moved J2 72.6 mm to (265.6, 66.4), turned to 180 degrees
- moved SW_BAT_01 63.2 mm to (260.6, 44.8), turned to 5 degrees
- moved S_MAT_20 23.9 mm to (36.0, 97.0)
- moved S_MAT_35 23.9 mm to (143.7, 141.2)
- moved FB_USB_01 23.9 mm to (153.0, 61.5)
- moved F_USB_02 23.9 mm to (139.0, 59.5)
- moved J_BAT_01 23.9 mm to (40.0, 49.5)
- moved J_USB_01 23.9 mm to (146.0, 58.9)
- moved R_USB_01 23.9 mm to (139.0, 57.0)
- moved R_USB_02 23.9 mm to (139.1, 58.0)
- moved S_MAT_00 23.9 mm to (36.0, 63.0)
- moved S_MAT_01 23.9 mm to (65.4, 53.0)
- moved S_MAT_02 23.9 mm to (90.7, 54.3)
- moved S_MAT_03 23.9 mm to (107.0, 63.1)
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Routing:
- net /Control_Board/GND: track 97.2 -> 93.9 mm
Other:
- board size 289.7 x 251.2 mm -> 285.8 x 230 mm
