File: pcb/control_board.kicad_sch (KiCad schematic)
At the start: 8 parts

Commit message: Work on PCBs.
Parts:
- added H1, H2, H3, H4, H5, H6: MountingHole_Pad, MountingHole:MountingHole_2.2mm_M2_Pad, symbol Mechanical:MountingHole_Pad
Connections:
- net 5V: now also J_VIK_OUT_DISP_01.6 (5V), J_VIK_OUT_INTC_01.6 (5V), J_VIK_OUT_SENS_01.6 (5V), J_VIK_OUT_SW_01.6 (5V)
- net GND: now also H1.1, H2.1, H3.1, H4.1, H5.1, H6.1
- net VEXT: now also J_VIK_OUT_DISP_01.5 (RGB_DO), J_VIK_OUT_INTC_01.5 (RGB_DO), J_VIK_OUT_SENS_01.5 (RGB_DO), J_VIK_OUT_SW_01.5 (RGB_DO); no longer J_VIK_OUT_DISP_01.6 (5V), J_VIK_OUT_INTC_01.6 (5V), J_VIK_OUT_SENS_01.6 (5V), J_VIK_OUT_SW_01.6 (5V)
- removed net RGB_DO1: J_VIK_OUT_DISP_01.5 (RGB_DO), J_VIK_OUT_SENS_01.5 (RGB_DO), J_VIK_OUT_SW_01.5 (RGB_DO), U_MCU_01.4 ([L]_P1.13)
- net RGB_DO2: no longer names the net of U_MCU_01.5 ([L]_P1.15)
- net RGB_DO2: no longer J_VIK_OUT_INTC_01.5 (RGB_DO)
- net RGB_DO3: no longer names the net of U_MCU_01.6 ([L]_A1_P0.03)
- no-connect marks 0 -> 9
