File: pcb/power_board.kicad_sch (KiCad schematic)
At the start: 10 parts

Commit message: Work on PCBs.
Parts:
- added H10, H11, H12, H7, H8, H9: MountingHole_Pad, MountingHole:MountingHole_2.2mm_M2_Pad, symbol Mechanical:MountingHole_Pad
- J_VIK_OUT_DISP_02: now not fitted; now left out of the parts list
Connections:
- net GP22 is gone; now on net BATT_MON: J_VIK_IN_INTC_01.4 (GP_AD2)
- net RGB_DO2 is gone; now on net VEXT: J_VIK_IN_INTC_01.8 (RGB_DO), J_VIK_OUT_DISP_02.5 (RGB_DO), J_VIK_OUT_SENS_02.5 (RGB_DO), J_VIK_OUT_SW_02.5 (RGB_DO)
- net 5V: now also J_VIK_IN_INTC_01.7 (5V), J_VIK_OUT_DISP_02.6 (5V), J_VIK_OUT_SENS_02.6 (5V), J_VIK_OUT_SW_02.6 (5V)
- net GND: now also H10.1, H11.1, H12.1, H7.1, H8.1, H9.1
- net VEXT: no longer J_VIK_IN_INTC_01.7 (5V), J_VIK_OUT_DISP_02.6 (5V), J_VIK_OUT_SENS_02.6 (5V), J_VIK_OUT_SW_02.6 (5V)
- net CS_SW2: no longer names the net of J_VIK_OUT_SW_02.10 (SPI_CS)
- net D+: no longer names the net of J_VIK_OUT_SW_02.9 (GP_AD2)
- net D-: no longer names the net of J_VIK_OUT_SW_02.7 (GP_AD1)
- net GP12: no longer names the net of J_VIK_OUT_SENS_02.9 (GP_AD2)
- no-connect marks 0 -> 4
