File: pcb/switch_board.kicad_sch (KiCad schematic)
At the start: 46 parts

Commit message: Work on PCBs.
Parts:
- added J1, J2: Conn_01x04, Connector_PinHeader_2.54mm:PinHeader_1x04_P2.54mm_Vertical, symbol Connector_Generic:Conn_01x04
- S_MAT_00, S_MAT_01, S_MAT_02, S_MAT_03, S_MAT_04, S_MAT_10, S_MAT_11, S_MAT_12, S_MAT_13, S_MAT_14, S_MAT_15, S_MAT_20, S_MAT_21, S_MAT_22, S_MAT_23, S_MAT_24, S_MAT_25, S_MAT_31, S_MAT_32, S_MAT_33, S_MAT_34, S_MAT_35: symbol Switch:SW_Push_45deg -> Switch:SW_Push_Shielded
- S_MAT_05, S_MAT_30: footprint (none) -> key-switches:SW_Kailh_Choc_V1V2_HotSwap_PTH_Double; symbol Switch:SW_Push_45deg -> Switch:SW_Push_Shielded
Connections:
- net RGB_DO1 is gone; now on net MOSI: J_VIK_IN_SW_01.5 (MOSI)
- net 5V: now also J_VIK_IN_SW_01.7 (5V)
- net D+: now also J_VIK_IN_SW_01.4 (GP_AD2); no longer J_VIK_IN_SW_01.9 (SCL)
- net D-: now also J_VIK_IN_SW_01.6 (GP_AD1); no longer J_VIK_IN_SW_01.7 (5V)
- net GND: now also J_BAT_01.1 (Pin_1), J_VIK_IN_SW_01.11 (GND), S_MAT_00.SH (B), S_MAT_01.SH (B), S_MAT_02.SH (B), S_MAT_03.SH (B), S_MAT_04.SH (B), S_MAT_05.SH (B), S_MAT_10.SH (B), S_MAT_11.SH (B), S_MAT_12.SH (B), S_MAT_13.SH (B), S_MAT_14.SH (B), S_MAT_15.SH (B), S_MAT_20.SH (B), S_MAT_21.SH (B), S_MAT_22.SH (B), S_MAT_23.SH (B), S_MAT_24.SH (B), S_MAT_25.SH (B), S_MAT_31.SH (B), S_MAT_32.SH (B), S_MAT_33.SH (B), S_MAT_34.SH (B), S_MAT_35.SH (B), J1.4 (Pin_4); no longer J_BAT_01.2 (Pin_2), J_VIK_IN_SW_01.2 (MISO), SW_RST_01.2
- net MISO: now also J_VIK_IN_SW_01.2 (MISO); no longer J_VIK_IN_SW_01.11 (GND)
- net MOSI: no longer J_VIK_IN_SW_01.8 (RGB_DO)
- net RST: now also J_VIK_IN_SW_01.3 (SPI_CS), J1.3 (Pin_3); no longer J_VIK_IN_SW_01.10 (SDA), SW_RST_01.1
- net SCL: now also J_VIK_IN_SW_01.9 (SCL); no longer J_VIK_IN_SW_01.4 (GP_AD2)
- net SCLK: now also J_VIK_IN_SW_01.1 (SCLK); no longer J_VIK_IN_SW_01.12 (3V3)
- net SDA: now also J_VIK_IN_SW_01.10 (SDA); no longer J_VIK_IN_SW_01.3 (SPI_CS)
- net VBAT: now also J1.2 (Pin_2); no longer SW_BAT_01.1 (A)
- net VDD: now also J_VIK_IN_SW_01.12 (3V3); no longer J_VIK_IN_SW_01.1 (SCLK)
- net VEXT: now also J_VIK_IN_SW_01.8 (RGB_DO); no longer J_VIK_IN_SW_01.6 (GP_AD1)
- net at SW_BAT_01.2 (B): now also J2.2 (Pin_2); no longer J_BAT_01.1 (Pin_1)
- net GNDPWR renamed SH
- net VBUS renamed VUSB
- new net: J1.1 (Pin_1), J_BAT_01.2 (Pin_2)
- new net: J2.1 (Pin_1), SW_BAT_01.1 (A)
- new net: J2.4 (Pin_4), SW_RST_01.2
- new net PLATE_GND: J2.3 (Pin_3), SW_RST_01.1
Other:
- moved on the sheet: J_BAT_01, SW_RST_01
