File: pcb/pcb_plate/pcb_plate.kicad_pcb (KiCad board)
At the start: 2 copper layers, 269.2 x 122.9 mm, 49 parts, among them J1 Conn_01x04, J2 Conn_01x04

Commit message: Redo matrix plates.
Parts:
- removed D_POW_01: 1N5819WS, Diode_SMD:D_SOD-323
- removed FB_USB_01: ~, Inductor_SMD:L_0805_2012Metric
- removed F_USB_02: SMD0805-050-16V, Fuse:Fuse_0805_2012Metric
- removed J1, J2: Conn_01x04, Connector_PinHeader_2.54mm:PinHeader_1x04_P2.54mm_Vertical
- removed J_BAT_01: Conn_01x02, Connector_JST:JST_GH_SM02B-GHS-TB_1x02-1MP_P1.25mm_Horizontal
- removed J_USB_01: USB_C_Receptacle_USB2.0_16P, Connector_USB:USB_C_Receptacle_HRO_TYPE-C-31-M-12
- removed J_VIK_IN_SW_01: vik-module-connector, vik:vik-module-connector-horizontal
- removed Q_POW_01: AO3401A, Package_TO_SOT_SMD:SOT-23
- removed R_MAT_01, R_MAT_02, R_MAT_11, R_MAT_12, R_MAT_21, R_MAT_22, R_MAT_31: 10K, Resistor_SMD:R_0201_0603Metric_Pad0.64x0.40mm_HandSolder
- removed R_POW_01: 100K, Resistor_SMD:R_0201_0603Metric_Pad0.64x0.40mm_HandSolder
- removed R_USB_01, R_USB_02: 5.1K, Resistor_SMD:R_0201_0603Metric_Pad0.64x0.40mm_HandSolder
- removed SW_BAT_01: SW_SPST, library:AS11CH
- removed SW_RST_01: SW_Push, Button_Switch_SMD:SW_Push_1P1T_NO_E-Switch_TL3301NxxxxxG
- removed S_MAT_00, S_MAT_01, S_MAT_02, S_MAT_03, S_MAT_04, S_MAT_10, S_MAT_11, S_MAT_12, S_MAT_13, S_MAT_14, S_MAT_15, S_MAT_20, S_MAT_21, S_MAT_22, S_MAT_23, S_MAT_24, S_MAT_25, S_MAT_31, S_MAT_32, S_MAT_33, S_MAT_34, S_MAT_35: SW_Push_45deg, key-switches:SW_Kailh_Choc_V1V2_HotSwap_PTH_Double
- removed U_MAT_01: MCP23017_SS, Package_SO:SSOP-28_5.3x10.2mm_P0.65mm
- removed U_POW_01: XC6220B331MR, Package_TO_SOT_SMD:SOT-23-5
- removed U_USB_01: SRV05-4, Package_TO_SOT_SMD:SOT-23-6
- added J_VIK_IN_SW_1: vik-module-connector, vik:vik-module-connector-horizontal, F.Cu at (140.8, 105.0)
- added J_VIK_IN_SW_2: vik-module-connector, vik:vik-module-connector-horizontal, F.Cu at (159.2, 105.0)
- added S_MAT_L00: SW_Push_45deg, key-switches:SW_GLP_Kailh_Choc_V1V2_HotSwap_PTH, F.Cu at (28.9, 42.8)
- added S_MAT_L01: SW_Push_45deg, key-switches:SW_GLP_Kailh_Choc_V1V2_HotSwap_PTH, F.Cu at (58.3, 32.9)
- added S_MAT_L02: SW_Push_45deg, key-switches:SW_GLP_Kailh_Choc_V1V2_HotSwap_PTH, F.Cu at (83.6, 34.2)
- added S_MAT_L03: SW_Push_45deg, key-switches:SW_GLP_Kailh_Choc_V1V2_HotSwap_PTH, F.Cu at (99.9, 42.9)
- added S_MAT_L04: SW_Push_45deg, key-switches:SW_GLP_Kailh_Choc_V1V2_HotSwap_PTH, F.Cu at (117.3, 47.6)
- added S_MAT_L10: SW_Push_45deg, key-switches:SW_GLP_Kailh_Choc_V1V2_HotSwap_PTH, F.Cu at (28.9, 59.8)
- added S_MAT_L11: SW_Push_45deg, key-switches:SW_GLP_Kailh_Choc_V1V2_HotSwap_PTH, F.Cu at (55.4, 49.6)
- added S_MAT_L12: SW_Push_45deg, key-switches:SW_GLP_Kailh_Choc_V1V2_HotSwap_PTH, F.Cu at (79.2, 50.6)
- added S_MAT_L13: SW_Push_45deg, key-switches:SW_GLP_Kailh_Choc_V1V2_HotSwap_PTH, F.Cu at (95.5, 59.4)
- added S_MAT_L14: SW_Push_45deg, key-switches:SW_GLP_Kailh_Choc_V1V2_HotSwap_PTH, F.Cu at (112.9, 64.0)
- added S_MAT_L15: SW_Push_45deg, key-switches:SW_GLP_Kailh_Choc_V1V2_HotSwap_PTH, F.Cu at (131.5, 94.7)
- added S_MAT_L20: SW_Push_45deg, key-switches:SW_GLP_Kailh_Choc_V1V2_HotSwap_PTH, F.Cu at (28.9, 76.8)
- added S_MAT_L21: SW_Push_45deg, key-switches:SW_GLP_Kailh_Choc_V1V2_HotSwap_PTH, F.Cu at (52.4, 66.3)
- added S_MAT_L22: SW_Push_45deg, key-switches:SW_GLP_Kailh_Choc_V1V2_HotSwap_PTH, F.Cu at (74.8, 67.0)
- added S_MAT_L23: SW_Push_45deg, key-switches:SW_GLP_Kailh_Choc_V1V2_HotSwap_PTH, F.Cu at (91.1, 75.8)
- added S_MAT_L24: SW_Push_45deg, key-switches:SW_GLP_Kailh_Choc_V1V2_HotSwap_PTH, F.Cu at (108.5, 80.4)
- added S_MAT_L25: SW_Push_45deg, key-switches:SW_GLP_Kailh_Choc_V1V2_HotSwap_PTH, F.Cu at (121.8, 108.5)
- added S_MAT_L31: SW_Push_45deg, key-switches:SW_GLP_Kailh_Choc_V1V2_HotSwap_PTH, F.Cu at (49.5, 83.1)
- added S_MAT_L32: SW_Push_45deg, key-switches:SW_GLP_Kailh_Choc_V1V2_HotSwap_PTH, F.Cu at (70.4, 83.4)
- added S_MAT_L33: SW_Push_45deg, key-switches:SW_GLP_Kailh_Choc_V1V2_HotSwap_PTH, F.Cu at (86.7, 92.2)
- added S_MAT_L34: SW_Push_45deg, key-switches:SW_GLP_Kailh_Choc_V1V2_HotSwap_PTH, F.Cu at (104.9, 98.9)
- added S_MAT_L35: SW_Push_45deg, key-switches:SW_GLP_Kailh_Choc_V1V2_HotSwap_PTH, F.Cu at (136.6, 121.0)
- added S_MAT_R00: SW_Push_45deg, key-switches:SW_GLP_Kailh_Choc_V1V2_HotSwap_PTH, F.Cu at (271.1, 42.9)
- added S_MAT_R01: SW_Push_45deg, key-switches:SW_GLP_Kailh_Choc_V1V2_HotSwap_PTH, F.Cu at (241.7, 32.9)
- added S_MAT_R02: SW_Push_45deg, key-switches:SW_GLP_Kailh_Choc_V1V2_HotSwap_PTH, F.Cu at (216.4, 34.2)
- added S_MAT_R03: SW_Push_45deg, key-switches:SW_GLP_Kailh_Choc_V1V2_HotSwap_PTH, F.Cu at (200.1, 43.0)
- added S_MAT_R04: SW_Push_45deg, key-switches:SW_GLP_Kailh_Choc_V1V2_HotSwap_PTH, F.Cu at (182.7, 47.6)
- added S_MAT_R10: SW_Push_45deg, key-switches:SW_GLP_Kailh_Choc_V1V2_HotSwap_PTH, F.Cu at (271.1, 59.8)
- added S_MAT_R11: SW_Push_45deg, key-switches:SW_GLP_Kailh_Choc_V1V2_HotSwap_PTH, F.Cu at (244.6, 49.6)
- added S_MAT_R12: SW_Push_45deg, key-switches:SW_GLP_Kailh_Choc_V1V2_HotSwap_PTH, F.Cu at (220.8, 50.6)
- added S_MAT_R13: SW_Push_45deg, key-switches:SW_GLP_Kailh_Choc_V1V2_HotSwap_PTH, F.Cu at (204.5, 59.3)
- added S_MAT_R14: SW_Push_45deg, key-switches:SW_GLP_Kailh_Choc_V1V2_HotSwap_PTH, F.Cu at (187.1, 64.0)
- added S_MAT_R15: SW_Push_45deg, key-switches:SW_GLP_Kailh_Choc_V1V2_HotSwap_PTH, F.Cu at (168.5, 94.7)
- added S_MAT_R20: SW_Push_45deg, key-switches:SW_GLP_Kailh_Choc_V1V2_HotSwap_PTH, F.Cu at (271.1, 76.8)
- added S_MAT_R21: SW_Push_45deg, key-switches:SW_GLP_Kailh_Choc_V1V2_HotSwap_PTH, F.Cu at (247.6, 66.4)
- added S_MAT_R22: SW_Push_45deg, key-switches:SW_GLP_Kailh_Choc_V1V2_HotSwap_PTH, F.Cu at (225.2, 67.1)
- added S_MAT_R23: SW_Push_45deg, key-switches:SW_GLP_Kailh_Choc_V1V2_HotSwap_PTH, F.Cu at (208.9, 75.8)
- added S_MAT_R24: SW_Push_45deg, key-switches:SW_GLP_Kailh_Choc_V1V2_HotSwap_PTH, F.Cu at (191.5, 80.5)
- added S_MAT_R25: SW_Push_45deg, key-switches:SW_GLP_Kailh_Choc_V1V2_HotSwap_PTH, F.Cu at (178.2, 108.6)
- added S_MAT_R31: SW_Push_45deg, key-switches:SW_GLP_Kailh_Choc_V1V2_HotSwap_PTH, F.Cu at (250.5, 83.1)
- added S_MAT_R32: SW_Push_45deg, key-switches:SW_GLP_Kailh_Choc_V1V2_HotSwap_PTH, F.Cu at (229.6, 83.5)
- added S_MAT_R33: SW_Push_45deg, key-switches:SW_GLP_Kailh_Choc_V1V2_HotSwap_PTH, F.Cu at (213.3, 92.2)
- added S_MAT_R34: SW_Push_45deg, key-switches:SW_GLP_Kailh_Choc_V1V2_HotSwap_PTH, F.Cu at (195.1, 98.9)
- added S_MAT_R35: SW_Push_45deg, key-switches:SW_GLP_Kailh_Choc_V1V2_HotSwap_PTH, F.Cu at (163.4, 121.1)
- moved REF** 1.19 mm to (151.0, 130.5)
- moved REF** 0.72 mm to (151.0, 111.0)
- moved REF** 0.72 mm to (151.0, 93.0)
Routing:
- net (no net): track 0.00 -> 534.5 mm
- net /Left/C0: track 0.00 -> 230.0 mm, vias 0 -> 1
- net /Left/R0: track 0.00 -> 213.5 mm
- net /Right/R0: track 0.00 -> 212.5 mm
- net /Left/C1: track 0.00 -> 210.9 mm, vias 0 -> 1
- net /Switch_Board/RST: track 207.6 -> 0.00 mm, vias 1 -> 0
- net /Left/R1: track 0.00 -> 205.6 mm
- net /Right/C2: track 0.00 -> 203.4 mm, vias 0 -> 1
- net /Right/C0: track 0.00 -> 198.8 mm, vias 0 -> 1
- net /Right/R1: track 0.00 -> 198.4 mm
- net /Right/C1: track 0.00 -> 195.0 mm, vias 0 -> 1
- net /Left/R2: track 0.00 -> 194.1 mm
- net /Right/R2: track 0.00 -> 191.2 mm
- net /Right/C3: track 0.00 -> 179.1 mm, vias 0 -> 1
- net /Right/R3: track 0.00 -> 177.9 mm
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- added copper zone on B.Cu, net /Left/GND
- added copper zone on F.Cu, net /Left/GND
- added copper zone on B.Cu, net /Right/GND
- added copper zone on F.Cu, net /Right/GND
- removed copper zone on B.Cu, net /Switch_Board/GND
- removed copper zone on F.Cu, net /Switch_Board/GND
- removed copper zone on B.Cu, net /Switch_Board/PLATE_GND
- removed copper zone on F.Cu, net /Switch_Board/PLATE_GND
Other:
- outline, holes or cut-outs redrawn
- board text added: "Matrix PCB"
- board text removed: "Main PCB"
- board text removed: "Switch Plate"
