File: pcb/pcb_plate/right.kicad_sch (KiCad schematic)
At the start: 0 parts

Commit message: Redo matrix plates.
Parts:
- added J_VIK_IN_SW_2: vik-module-connector, vik:vik-module-connector-horizontal, symbol vik:vik-module-connector
- added S_MAT_R00, S_MAT_R01, S_MAT_R02, S_MAT_R03, S_MAT_R04, S_MAT_R10, S_MAT_R11, S_MAT_R12, S_MAT_R13, S_MAT_R14, S_MAT_R15, S_MAT_R20, S_MAT_R21, S_MAT_R22, S_MAT_R23, S_MAT_R24, S_MAT_R25, S_MAT_R31, S_MAT_R32, S_MAT_R33, S_MAT_R34, S_MAT_R35: SW_Push_45deg, key-switches:SW_GLP_Kailh_Choc_V1V2_HotSwap_PTH, symbol Switch:SW_Push_45deg
Connections:
- new net C0: J_VIK_IN_SW_2.10 (SDA), S_MAT_R00.1, S_MAT_R10.1, S_MAT_R20.1
- new net C1: J_VIK_IN_SW_2.9 (SCL), S_MAT_R01.1, S_MAT_R11.1, S_MAT_R21.1, S_MAT_R31.1
- new net C2: J_VIK_IN_SW_2.8 (RGB_DO), S_MAT_R02.1, S_MAT_R12.1, S_MAT_R22.1, S_MAT_R32.1
- new net C3: J_VIK_IN_SW_2.7 (5V), S_MAT_R03.1, S_MAT_R13.1, S_MAT_R23.1, S_MAT_R33.1
- new net C4: J_VIK_IN_SW_2.6 (GP_AD1), S_MAT_R04.1, S_MAT_R14.1, S_MAT_R24.1, S_MAT_R34.1
- new net C5: J_VIK_IN_SW_2.5 (MOSI), S_MAT_R15.1, S_MAT_R25.1, S_MAT_R35.1
- new net GND: J_VIK_IN_SW_2.11 (GND)
- new net R0: J_VIK_IN_SW_2.4 (GP_AD2), S_MAT_R00.2, S_MAT_R01.2, S_MAT_R02.2, S_MAT_R03.2, S_MAT_R04.2
- new net R1: J_VIK_IN_SW_2.3 (SPI_CS), S_MAT_R10.2, S_MAT_R11.2, S_MAT_R12.2, S_MAT_R13.2, S_MAT_R14.2, S_MAT_R15.2
- new net R2: J_VIK_IN_SW_2.2 (MISO), S_MAT_R20.2, S_MAT_R21.2, S_MAT_R22.2, S_MAT_R23.2, S_MAT_R24.2, S_MAT_R25.2
- new net R3: J_VIK_IN_SW_2.1 (SCLK), S_MAT_R31.2, S_MAT_R32.2, S_MAT_R33.2, S_MAT_R34.2, S_MAT_R35.2
- new net VDD: J_VIK_IN_SW_2.12 (3V3)
