File: pcb/matrix_plate/left.kicad_sch (KiCad schematic)
At the start: 23 parts

Commit message: Work on PCBs.
Parts:
- added R_MAT_13, R_MAT_14, R_MAT_23, R_MAT_24, R_MAT_3, R_MAT_32, R_MAT_4: 10K, Resistor_SMD:R_0201_0603Metric_Pad0.64x0.40mm_HandSolder, symbol Device:R
- added U_MAT_2: MCP23017_SS, Package_SO:SSOP-28_5.3x10.2mm_P0.65mm, symbol Interface_Expansion:MCP23017x-x-SS
Connections:
- net C0: now also U_MAT_2.1 (GPB0); no longer J_VIK_IN_SW_1.10 (SDA)
- net C1: now also U_MAT_2.2 (GPB1); no longer J_VIK_IN_SW_1.9 (SCL)
- net C2: now also U_MAT_2.3 (GPB2); no longer J_VIK_IN_SW_1.8 (RGB_DO)
- net C3: now also U_MAT_2.4 (GPB3); no longer J_VIK_IN_SW_1.7 (5V)
- net C4: now also U_MAT_2.5 (GPB4); no longer J_VIK_IN_SW_1.6 (GP_AD1)
- net C5: now also U_MAT_2.6 (GPB5); no longer J_VIK_IN_SW_1.5 (MOSI)
- net GND: now also J_VIK_IN_SW_1.13 (MP), J_VIK_IN_SW_1.14 (MP), R_MAT_14.2, R_MAT_24.2, R_MAT_4.2, U_MAT_2.10 (V_{SS})
- net R0: now also U_MAT_2.21 (GPA0); no longer J_VIK_IN_SW_1.4 (GP_AD2)
- net R1: now also U_MAT_2.22 (GPA1); no longer J_VIK_IN_SW_1.3 (SPI_CS)
- net R2: now also U_MAT_2.23 (GPA2); no longer J_VIK_IN_SW_1.2 (MISO)
- net R3: now also U_MAT_2.24 (GPA3); no longer J_VIK_IN_SW_1.1 (SCLK)
- net VDD: now also R_MAT_13.1, R_MAT_23.1, R_MAT_3.1, R_MAT_32.1, U_MAT_2.9 (V_{DD})
- new net: R_MAT_13.2, R_MAT_14.1, U_MAT_2.16 (A1)
- new net: R_MAT_3.2, R_MAT_4.1, U_MAT_2.15 (A0)
- new net: R_MAT_23.2, R_MAT_24.1, U_MAT_2.17 (A2)
- new net: R_MAT_32.2, U_MAT_2.18 (~{RESET})
- new net SCL: J_VIK_IN_SW_1.9 (SCL), U_MAT_2.13 (SDA)
- new net SDA: J_VIK_IN_SW_1.10 (SDA), U_MAT_2.12 (SCK)
- no-connect marks 0 -> 16
Other:
- moved on the sheet: S_MAT_L00, S_MAT_L01, S_MAT_L02, S_MAT_L03, S_MAT_L04, S_MAT_L10, S_MAT_L11, S_MAT_L12, S_MAT_L13, S_MAT_L14, S_MAT_L15, S_MAT_L20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

Commit message: Tentatively finish PCBs.
Parts:
- added SW_RST_1: SW_Push, Button_Switch_THT:SW_PUSH_6mm, symbol Switch:SW_Push
- R_MAT_13, R_MAT_14, R_MAT_23, R_MAT_24, R_MAT_3, R_MAT_32, R_MAT_4: footprint Resistor_SMD:R_0201_0603Metric_Pad0.64x0.40mm_HandSolder -> Resistor_SMD:R_1206_3216Metric_Pad1.30x1.75mm_HandSolder
Connections:
- net GND: now also SW_RST_1.2
- net RST: now reaches J_VIK_IN_SW_1.6 (GP_AD1)
- net RST: now also SW_RST_1.1
- no-connect marks 16 -> 15
Changed lines of the file:
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@@
 	)
 	(no_connect
-		(at 293.37 40.64)
-	)
-	(no_connect
 		(at 293.37 27.94)
 	)
@@
 		)
 	)
+	(label "RST"
+		(at 337.82 35.56 180)
+		(effects
+			(font
+				(size 1.27 1.27)
+			)
+			(justify right bottom)
+		)
+	)
+	(label "GND"
+		(at 347.98 35.56 0)
+		(effects
+			(font
+				(size 1.27 1.27)
+			)
+			(justify left bottom)
+		)
+	)
 	(label "R1"
 		(at 87.63 38.1 0)
@@
 		)
 	)
+	(label "RST"
+		(at 293.37 40.64 180)
+		(effects
+			(font
+				(size 1.27 1.27)
+			)
+			(justify right bottom)
+		)
+	)
 	(label "C2"
 		(at 189.23 25.4 90)
@@
 			)
 		)
-		(property "Footprint" "Resistor_SMD:R_0201_0603Metric_Pad0.64x0.40mm_HandSolder"
+		(property "Footprint" "Resistor_SMD:R_1206_3216Metric_Pad1.30x1.75mm_HandSolder"
 			(at 35.56 71.882 90)
 			(hide yes)
@@
 	)
 	(symbol
+		(lib_id "Switch:SW_Push")
+		(at 342.9 35.56 0)
+		(unit 1)
+		(body_style 1)
+		(exclude_from_sim no)
+		(in_bom yes)
+		(on_board yes)
+		(in_pos_files yes)
+		(dnp no)
+		(fields_autoplaced yes)
+		(property "Reference" "SW_RST_1"
+			(at 342.9 27.94 0)
+			(show_name no)
+			(do_not_autoplace no)
+			(effects
+				(font
+					(size 1.27 1.27)
+				)
+			)
+		)
+		(property "Value" "SW_Push"
+			(at 342.9 30.48 0)
+			(show_name no)
+			(do_not_autoplace no)
+			(effects
+				(font
+					(size 1.27 1.27)
+				)
+			)
+		)
+		(property "Footprint" "Button_Switch_THT:SW_PUSH_6mm"
+			(at 342.9 30.48 0)
+			(show_name no)
+			(do_not_autoplace no)
+			(effects
+				(font
+					(size 1.27 1.27)
+				)
+			)
+		)
+		(property "Datasheet" ""
+			(at 342.9 30.48 0)
+			(hide yes)
+			(show_name no)
+			(do_not_autoplace no)
+			(effects
+				(font
+					(size 1.27 1.27)
+				)
+			)
+		)
+		(property "Description" "Push button switch, generic, two pins"
+			(at 342.9 35.56 0)
+			(hide yes)
+			(show_name no)
+			(do_not_autoplace no)
+			(effects
+				(font
+					(size 1.27 1.27)
+				)
+			)
+		)
+		(pin "2"
+		)
+		(pin "1"
+		)
+		(instances
+			(project "matrix_plate"
+				(path "/ff6e9c14-03d1-4298-be5c-ff86cb590acc/417aa41b-7daf-492f-bffc-85846200bac5"
+					(reference "SW_RST_1")
+					(unit 1)
+				)
+			)
+		)
+	)
+	(symbol
 		(lib_id "Switch:SW_Push_45deg")
 		(at 209.55 68.58 0)
@@
 			)
 		)
-		(property "Footprint" "Resistor_SMD:R_0201_0603Metric_Pad0.64x0.40mm_HandSolder"
+		(property "Footprint" "Resistor_SMD:R_1206_3216Metric_Pad1.30x1.75mm_HandSolder"
 			(at 53.34 72.898 90)
 			(hide yes)
@@
 			)
 		)
-		(property "Footprint" "Resistor_SMD:R_0201_0603Metric_Pad0.64x0.40mm_HandSolder"
+		(property "Footprint" "Resistor_SMD:R_1206_3216Metric_Pad1.30x1.75mm_HandSolder"
 			(at 55.88 57.658 90)
 			(hide yes)
@@
 			)
 		)
-		(property "Footprint" "Resistor_SMD:R_0201_0603Metric_Pad0.64x0.40mm_HandSolder"
+		(property "Footprint" "Resistor_SMD:R_1206_3216Metric_Pad1.30x1.75mm_HandSolder"
 			(at 56.642 81.28 90)
 			(hide yes)
@@
 			)
 		)
-		(property "Footprint" "Resistor_SMD:R_0201_0603Metric_Pad0.64x0.40mm_HandSolder"
+		(property "Footprint" "Resistor_SMD:R_1206_3216Metric_Pad1.30x1.75mm_HandSolder"
 			(at 56.642 66.04 90)
 			(hide yes)
@@
 			)
 		)
-		(property "Footprint" "Resistor_SMD:R_0201_0603Metric_Pad0.64x0.40mm_HandSolder"
+		(property "Footprint" "Resistor_SMD:R_1206_3216Metric_Pad1.30x1.75mm_HandSolder"
 			(at 53.34 74.422 90)
 			(hide yes)
@@
 			)
 		)
-		(property "Footprint" "Resistor_SMD:R_0201_0603Metric_Pad0.64x0.40mm_HandSolder"
+		(property "Footprint" "Resistor_SMD:R_1206_3216Metric_Pad1.30x1.75mm_HandSolder"
 			(at 38.862 78.74 90)
 			(hide yes)
