File: pcb/matrix_plate/matrix_plate.kicad_pcb (KiCad board)
At the start: 2 copper layers, 269.2 x 122.9 mm, 49 parts

Commit message: Work on PCBs.
Parts:
- added FB_USB_1: ~, Inductor_SMD:L_0805_2012Metric, B.Cu at (168.5, 38.5)
- added F_USB_2: SMD0805-050-16V, Fuse:Fuse_0805_2012Metric, B.Cu at (168.5, 43.4)
- added J_USB_1: USB_C_Receptacle_USB2.0_16P, Connector_USB:USB_C_Receptacle_HRO_TYPE-C-31-M-12, F.Cu at (161.0, 39.2)
- added R_MAT_13: 10K, Resistor_SMD:R_0201_0603Metric_Pad0.64x0.40mm_HandSolder, F.Cu at (38.0, 28.4)
- added R_MAT_14: 10K, Resistor_SMD:R_0201_0603Metric_Pad0.64x0.40mm_HandSolder, F.Cu at (38.0, 25.6)
- added R_MAT_15: 10K, Resistor_SMD:R_0201_0603Metric_Pad0.64x0.40mm_HandSolder, F.Cu at (253.5, 26.9)
- added R_MAT_16: 10K, Resistor_SMD:R_0201_0603Metric_Pad0.64x0.40mm_HandSolder, F.Cu at (253.5, 24.1)
- added R_MAT_23: 10K, Resistor_SMD:R_0201_0603Metric_Pad0.64x0.40mm_HandSolder, F.Cu at (39.0, 28.4)
- added R_MAT_24: 10K, Resistor_SMD:R_0201_0603Metric_Pad0.64x0.40mm_HandSolder, F.Cu at (39.0, 25.6)
- added R_MAT_25: 10K, Resistor_SMD:R_0201_0603Metric_Pad0.64x0.40mm_HandSolder, F.Cu at (254.5, 26.9)
- added R_MAT_26: 10K, Resistor_SMD:R_0201_0603Metric_Pad0.64x0.40mm_HandSolder, F.Cu at (254.5, 24.1)
- added R_MAT_3: 10K, Resistor_SMD:R_0201_0603Metric_Pad0.64x0.40mm_HandSolder, F.Cu at (37.0, 28.4)
- added R_MAT_32: 10K, Resistor_SMD:R_0201_0603Metric_Pad0.64x0.40mm_HandSolder, F.Cu at (40.0, 28.4)
- added R_MAT_33: 10K, Resistor_SMD:R_0201_0603Metric_Pad0.64x0.40mm_HandSolder, F.Cu at (255.5, 26.9)
- added R_MAT_4: 10K, Resistor_SMD:R_0201_0603Metric_Pad0.64x0.40mm_HandSolder, F.Cu at (37.0, 25.6)
- added R_MAT_5: 10K, Resistor_SMD:R_0201_0603Metric_Pad0.64x0.40mm_HandSolder, F.Cu at (252.5, 26.9)
- added R_MAT_6: 10K, Resistor_SMD:R_0201_0603Metric_Pad0.64x0.40mm_HandSolder, F.Cu at (252.5, 24.0)
- added R_USB_1: 5.1K, Resistor_SMD:R_0201_0603Metric_Pad0.64x0.40mm_HandSolder, B.Cu at (154.4, 39.8)
- added R_USB_2: 5.1K, Resistor_SMD:R_0201_0603Metric_Pad0.64x0.40mm_HandSolder, B.Cu at (154.4, 40.5)
- added U_MAT_2: MCP23017_SS, Package_SO:SSOP-28_5.3x10.2mm_P0.65mm, B.Cu at (41.9, 29.0)
- added U_MAT_3: MCP23017_SS, Package_SO:SSOP-28_5.3x10.2mm_P0.65mm, B.Cu at (257.3, 27.5)
Connections:
- J_VIK_IN_SW_1 pad 1: /Left/R3 -> unconnected-(J_VIK_IN_SW_1-SCLK-Pad1)
- J_VIK_IN_SW_1 pad 10: /Left/C0 -> /Left/SDA
- J_VIK_IN_SW_1 pad 2: /Left/R2 -> unconnected-(J_VIK_IN_SW_1-MISO-Pad2)
- J_VIK_IN_SW_1 pad 3: /Left/R1 -> unconnected-(J_VIK_IN_SW_1-SPI_CS-Pad3)
- J_VIK_IN_SW_1 pad 4: /Left/R0 -> unconnected-(J_VIK_IN_SW_1-GP_AD2-Pad4)
- J_VIK_IN_SW_1 pad 5: /Left/C5 -> unconnected-(J_VIK_IN_SW_1-MOSI-Pad5)
- J_VIK_IN_SW_1 pad 6: /Left/C4 -> unconnected-(J_VIK_IN_SW_1-GP_AD1-Pad6)
- J_VIK_IN_SW_1 pad 7: /Left/C3 -> unconnected-(J_VIK_IN_SW_1-5V-Pad7)
- J_VIK_IN_SW_1 pad 8: /Left/C2 -> unconnected-(J_VIK_IN_SW_1-RGB_DO-Pad8)
- J_VIK_IN_SW_1 pad 9: /Left/C1 -> /Left/SCL
- J_VIK_IN_SW_2 pad 1: /Right/R3 -> unconnected-(J_VIK_IN_SW_2-SCLK-Pad1)
- J_VIK_IN_SW_2 pad 10: /Right/C0 -> /Right/SDA
- J_VIK_IN_SW_2 pad 2: /Right/R2 -> unconnected-(J_VIK_IN_SW_2-MISO-Pad2)
- J_VIK_IN_SW_2 pad 3: /Right/R1 -> unconnected-(J_VIK_IN_SW_2-SPI_CS-Pad3)
- J_VIK_IN_SW_2 pad 4: /Right/R0 -> /Right/D+
- J_VIK_IN_SW_2 pad 5: /Right/C5 -> unconnected-(J_VIK_IN_SW_2-MOSI-Pad5)
- J_VIK_IN_SW_2 pad 6: /Right/C4 -> /Right/D-
- J_VIK_IN_SW_2 pad 7: /Right/C3 -> /Right/VUSB
- J_VIK_IN_SW_2 pad 8: /Right/C2 -> unconnected-(J_VIK_IN_SW_2-RGB_DO-Pad8)
- J_VIK_IN_SW_2 pad 9: /Right/C1 -> /Right/SCL
Routing:
- net /Right/VDD: track 0.00 -> 173.6 mm, vias 0 -> 1
- net /Left/C0: track 230.0 -> 58.5 mm, vias 1 -> 0
- net /Left/SCL: track 0.00 -> 171.4 mm, vias 0 -> 1
- net /Left/SDA: track 0.00 -> 169.0 mm, vias 0 -> 1
- net /Left/VDD: track 0.00 -> 167.6 mm, vias 0 -> 2
- net /Right/SDA: track 0.00 -> 163.4 mm, vias 0 -> 1
- net /Right/SCL: track 0.00 -> 162.0 mm, vias 0 -> 1
- net /Left/C5: track 53.3 -> 210.7 mm, vias 1 -> 0
- net /Right/C0: track 198.8 -> 71.0 mm, vias 1 -> 0
- net /Right/C1: track 195.0 -> 70.9 mm, vias 1 -> 0
- net /Left/C1: track 210.9 -> 97.0 mm, vias 1 -> 0
- net /Right/C5: track 85.9 -> 192.8 mm, vias 1 -> 0
- net /Right/C2: track 203.4 -> 110.8 mm, vias 1 -> 0
- net /Left/R3: track 161.3 -> 247.6 mm, vias 0 -> 1
- net /Right/D-: track 0.00 -> 82.9 mm
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
Commit message: Tentatively finish PCBs.
Parts:
- added D2: LED_ARGB, LED_SMD:LED_Kingbright_APFA3010_3x1.5mm_Horizontal, F.Cu at (180.5, 89.5)
- added R2: 470, Resistor_SMD:R_1206_3216Metric_Pad1.30x1.75mm_HandSolder, F.Cu at (180.5, 83.5)
- added R3: 330, Resistor_SMD:R_1206_3216Metric_Pad1.30x1.75mm_HandSolder, F.Cu at (177.5, 79.5)
- added R4: 270, Resistor_SMD:R_1206_3216Metric_Pad1.30x1.75mm_HandSolder, F.Cu at (179.0, 81.5)
- added SW_RST_1: SW_Push, Button_Switch_THT:SW_PUSH_6mm, F.Cu at (121.1, 78.8)
- FB_USB_1: footprint Inductor_SMD:L_0805_2012Metric -> Inductor_SMD:L_1206_3216Metric_Pad1.22x1.90mm_HandSolder
- F_USB_2: footprint Fuse:Fuse_0805_2012Metric -> Fuse:Fuse_1206_3216Metric_Pad1.42x1.75mm_HandSolder
- R_MAT_13, R_MAT_14, R_MAT_15, R_MAT_16, R_MAT_23, R_MAT_24, R_MAT_25, R_MAT_26, R_MAT_3, R_MAT_32, R_MAT_33, R_MAT_4, R_MAT_5, R_MAT_6, R_USB_1, R_USB_2: footprint Resistor_SMD:R_0201_0603Metric_Pad0.64x0.40mm_HandSolder -> Resistor_SMD:R_1206_3216Metric_Pad1.30x1.75mm_HandSolder
- moved R_MAT_4 11.7 mm to (48.0, 21.5), turned to 0 degrees
- moved R_MAT_14 10.1 mm to (48.0, 24.0), turned to 0 degrees
- moved R_MAT_24 9.05 mm to (48.0, 26.5), turned to 0 degrees
- moved R_MAT_33 7.96 mm to (260.0, 33.5)
- moved R_MAT_25 7.24 mm to (257.5, 33.5)
- moved R_MAT_15 6.74 mm to (255.0, 33.5)
- moved R_MAT_5 6.59 mm to (252.5, 33.5)
- moved R_MAT_32 6.54 mm to (46.0, 31.0)
- moved R_MAT_23 5.19 mm to (43.5, 31.0)
- moved R_MAT_13 3.96 mm to (41.0, 31.0)
- moved R_MAT_3 2.97 mm to (38.5, 31.0)
- moved R_USB_1 2.95 mm to (152.5, 42.0), turned to -90 degrees
- moved R_MAT_26 2.19 mm to (256.0, 22.5)
- moved R_MAT_6 2.12 mm to (251.0, 22.5)
- moved R_USB_2 1.61 mm to (155.0, 42.0), turned to -90 degrees
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Connections:
- J_VIK_IN_SW_1 pad 6: unconnected-(J_VIK_IN_SW_1-GP_AD1-Pad6) -> /Left/RST
- J_VIK_IN_SW_2 pad 8: unconnected-(J_VIK_IN_SW_2-RGB_DO-Pad8) -> /Right/CHG_STAT
- U_MAT_3 pad 25: unconnected-(U_MAT_3-GPA4-Pad25) -> /Right/CHG_STAT
Routing:
- net /Right/CHG_STAT: track 0.00 -> 234.2 mm, vias 0 -> 1
- net /Left/RST: track 0.00 -> 36.2 mm
- net /Right/VUSB: track 69.8 -> 83.6 mm, vias 1 -> 2
- net Net-(U_MAT_2-A0): track 3.82 -> 16.4 mm
- net (no net): track 534.5 -> 522.4 mm
- net /Left/VDD: track 167.6 -> 179.4 mm, vias 2 -> 1
- net /Left/R0: track 169.2 -> 157.6 mm
- net Net-(U_MAT_2-A2): track 3.55 -> 14.6 mm
- net Net-(U_MAT_2-A1): track 3.65 -> 14.7 mm
- net Net-(D2-GA): track 0.00 -> 10.7 mm
- net /Left/R3: track 247.6 -> 238.1 mm
- net Net-(U_MAT_3-A0): track 3.82 -> 12.4 mm
- net Net-(D2-BA): track 0.00 -> 8.04 mm
- net /Right/R2: track 234.6 -> 226.8 mm
- net Net-(U_MAT_3-A2): track 3.56 -> 11.4 mm
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