File: pcb/matrix_plate/matrix_plate.kicad_pcb (KiCad board)
At the start: 2 copper layers, 269.2 x 122.9 mm, 75 parts

Commit message: Rework PCBs to ensure adequate clearance between them.
Parts:
- U_MAT_2, U_MAT_3: moved to F.Cu
- moved R_MAT_4 34.0 mm to (40.0, 54.5), turned to 180 degrees
- moved R_MAT_26 31.8 mm to (260.1, 54.0), turned to 0 degrees
- moved R_MAT_16 29.7 mm to (260.1, 51.5), turned to 0 degrees
- moved R_MAT_14 29.1 mm to (40.0, 52.0), turned to 180 degrees
- moved R_MAT_6 28.0 mm to (260.1, 49.0), turned to 0 degrees
- moved R_MAT_24 24.4 mm to (40.0, 49.5), turned to 180 degrees
- moved R_MAT_32 17.1 mm to (40.0, 47.0), turned to 0 degrees
- moved R_MAT_5 14.6 mm to (260.0, 46.0), turned to 180 degrees
- moved R_MAT_23 13.9 mm to (40.0, 44.5), turned to 0 degrees
- moved R_MAT_15 11.2 mm to (260.0, 43.5), turned to 180 degrees
- moved R_MAT_13 11.0 mm to (40.0, 42.0), turned to 0 degrees
- moved R_MAT_3 8.63 mm to (40.0, 39.5), turned to 0 degrees
- moved R_MAT_25 7.91 mm to (260.0, 41.0), turned to 180 degrees
- moved R_MAT_33 5.00 mm to (260.0, 38.5), turned to 180 degrees
- turned U_MAT_2 to -90 degrees
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Routing:
- net /Left/R0: track 157.6 -> 139.9 mm, vias 1 -> 0
- net Net-(U_MAT_3-A2): track 11.4 -> 25.8 mm, vias 1 -> 0
- net Net-(U_MAT_3-A1): track 10.8 -> 23.3 mm, vias 1 -> 0
- net Net-(U_MAT_2-A0): track 16.4 -> 25.1 mm, vias 1 -> 0
- net /Right/C2: track 111.4 -> 103.0 mm, vias 0 -> 1
- net Net-(U_MAT_2-~{RESET}): track 8.68 -> 16.8 mm, vias 1 -> 0
- net Net-(U_MAT_2-A1): track 14.7 -> 22.8 mm, vias 1 -> 0
- net /Right/C5: track 193.2 -> 185.2 mm, vias 0 -> 1
- net /Right/R0: track 160.4 -> 152.4 mm, vias 1 -> 0
- net Net-(U_MAT_3-A0): track 12.4 -> 20.3 mm, vias 1 -> 0
- net /Right/VDD: track 180.2 -> 188.0 mm, vias 1 -> 2
- net /Left/C0: track 58.5 -> 66.2 mm, vias 0 -> 1
- net /Right/C1: track 70.9 -> 78.2 mm, vias 0 -> 1
- net /Right/C3: track 139.1 -> 131.9 mm, vias 0 -> 1
- net /Right/C4: track 151.9 -> 145.0 mm, vias 0 -> 1
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