File: pcb/matrix_plate/matrix_plate.kicad_pcb (KiCad board)
At the start: 2 copper layers, 269.2 x 122.9 mm, 75 parts

Commit message: Add I2C pull-ups to matrix plates.
Parts:
- added R_MAT_34: 10K, Resistor_SMD:R_1206_3216Metric_Pad1.30x1.75mm_HandSolder, F.Cu at (40.0, 49.5)
- added R_MAT_35: 10K, Resistor_SMD:R_1206_3216Metric_Pad1.30x1.75mm_HandSolder, F.Cu at (40.0, 52.0)
- added R_MAT_36: 10K, Resistor_SMD:R_1206_3216Metric_Pad1.30x1.75mm_HandSolder, F.Cu at (260.0, 48.5)
- added R_MAT_37: 10K, Resistor_SMD:R_1206_3216Metric_Pad1.30x1.75mm_HandSolder, F.Cu at (260.0, 51.0)
- moved R_MAT_14 5.35 mm to (40.0, 57.4)
- moved R_MAT_24 5.35 mm to (40.0, 54.9)
- moved R_MAT_4 5.35 mm to (40.0, 59.9)
- moved R_MAT_16 4.50 mm to (260.1, 56.0)
- moved R_MAT_26 4.50 mm to (260.1, 58.5)
- moved R_MAT_6 4.50 mm to (260.1, 53.5)
Routing:
- net /Left/SCL: track 168.7 -> 201.1 mm, vias 0 -> 2
- net /Left/SDA: track 166.5 -> 194.5 mm, vias 0 -> 2
- net /Right/SCL: track 160.8 -> 188.8 mm, vias 0 -> 2
- net /Right/SDA: track 161.7 -> 186.7 mm, vias 0 -> 2
- net Net-(U_MAT_2-A0): track 25.1 -> 30.4 mm
- net Net-(U_MAT_2-A2): track 20.0 -> 25.3 mm
- net Net-(U_MAT_2-A1): track 22.8 -> 28.1 mm
- net Net-(U_MAT_3-A0): track 20.3 -> 25.6 mm
- net /Right/VDD: track 188.0 -> 193.0 mm
- net /Left/VDD: track 181.8 -> 186.7 mm
- net Net-(U_MAT_3-A2): track 25.8 -> 30.6 mm
- net Net-(U_MAT_3-A1): track 23.3 -> 28.1 mm
- net /Left/R1: track 226.8 -> 231.5 mm
- net /Right/R1: track 223.7 -> 225.3 mm
- net /Right/GND: vias 36 -> 38
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
Commit message: Move all components to top of matrix plate to improve manufacturability.
Parts:
- FB_USB_1, F_USB_2, R_USB_1, R_USB_2: moved to F.Cu
- moved R_USB_1 29.9 mm to (175.0, 61.8), turned to 0 degrees
- moved R_USB_2 29.9 mm to (175.0, 64.2), turned to 0 degrees
- moved FB_USB_1 29.0 mm to (175.0, 66.8)
- moved F_USB_2 26.7 mm to (175.0, 69.2)
Routing:
- net Net-(J_USB_1-CC2): track 6.60 -> 41.5 mm, vias 1 -> 0
- net /Right/SH: track 18.2 -> 48.9 mm
- net /Right/VUSB_RAW: track 8.28 -> 37.6 mm, vias 2 -> 3
- net /Right/VUSB: track 83.6 -> 61.7 mm, vias 2 -> 3
- net /Right/GND: track 29.5 -> 45.0 mm, vias 38 -> 40
- net Net-(J_USB_1-CC1): track 13.4 -> 28.3 mm, vias 1 -> 2
- net /Right/CHG_STAT: track 230.8 -> 241.1 mm
- net /Right/VDD: track 193.0 -> 196.4 mm
- net /Right/SCL: track 188.8 -> 192.1 mm
- net /Right/SDA: track 186.7 -> 190.0 mm

Commit message: Standardize on 0805 footprint for passive components.
Parts:
- FB_USB_1: footprint Inductor_SMD:L_1206_3216Metric_Pad1.22x1.90mm_HandSolder -> Inductor_SMD:L_0805_2012Metric_Pad1.05x1.20mm_HandSolder
- F_USB_2: footprint Fuse:Fuse_1206_3216Metric_Pad1.42x1.75mm_HandSolder -> Fuse:Fuse_0805_2012Metric_Pad1.15x1.40mm_HandSolder
- R2, R3, R4, R_MAT_13, R_MAT_14, R_MAT_15, R_MAT_16, R_MAT_23, R_MAT_24, R_MAT_25, R_MAT_26, R_MAT_3, R_MAT_32, R_MAT_33, R_MAT_34, R_MAT_35, R_MAT_36, R_MAT_37, R_MAT_4, R_MAT_5, R_MAT_6, R_USB_1, R_USB_2: footprint Resistor_SMD:R_1206_3216Metric_Pad1.30x1.75mm_HandSolder -> Resistor_SMD:R_0805_2012Metric_Pad1.20x1.40mm_HandSolder
- SW_RST_1: footprint Button_Switch_THT:SW_PUSH_6mm -> Button_Switch_SMD:SW_Push_1P1T_NO_E-Switch_TL3301NxxxxxG
- moved SW_RST_1 5.32 mm to (122.0, 84.0), turned to -115 degrees
Routing:
- net Net-(U_MAT_3-~{RESET}): track 8.93 -> 14.6 mm
- net /Right/GND: track 45.0 -> 50.1 mm
- net /Left/RST: track 36.2 -> 34.1 mm
- net /Left/C0: track 66.2 -> 64.5 mm
- net /Left/R1: track 231.5 -> 233.1 mm
- net Net-(U_MAT_2-A2): track 25.3 -> 24.4 mm, vias 0 -> 2
- net /Right/SDA: track 190.0 -> 190.9 mm
- net Net-(U_MAT_2-A0): track 30.4 -> 29.6 mm
- net Net-(U_MAT_3-A0): track 25.6 -> 25.0 mm, vias 0 -> 2
- net /Right/VUSB: track 61.7 -> 61.2 mm
- net Net-(J_USB_1-CC1): track 28.3 -> 28.9 mm
- net Net-(U_MAT_2-A1): track 28.1 -> 27.6 mm, vias 0 -> 2
- net Net-(U_MAT_3-A1): track 28.1 -> 27.7 mm, vias 0 -> 2
- net /Left/GND: vias 26 -> 28

Commit message: Move diodes to front of matrix plates for cheaper assembly.
Parts:
- removed R_MAT_13, R_MAT_15, R_MAT_23, R_MAT_25, R_MAT_3, R_MAT_6: 10K, Resistor_SMD:R_0805_2012Metric_Pad1.20x1.40mm_HandSolder
- moved R_L_A0 10.1 mm to (42.0, 50.0)
- moved R_L_A1 10.1 mm to (42.0, 47.5), turned to 0 degrees
- moved R_L_A2 10.1 mm to (42.0, 45.0), turned to 0 degrees
- moved R_L_RST_1 10.1 mm to (42.0, 37.1)
- moved R_L_SCL_1 10.1 mm to (42.0, 42.1)
- moved R_L_SDA_1 10.1 mm to (42.0, 39.6)
- moved R_R_A1 7.50 mm to (260.0, 48.5)
- moved R_R_A2 7.50 mm to (260.0, 51.0)
- moved R_R_A0 5.00 mm to (260.0, 41.0)
- moved R_R_SCL_1 5.00 mm to (260.0, 46.0)
- moved R_R_SDA_1 5.00 mm to (260.0, 43.5)
- moved SW_RST_1 1.12 mm to (123.0, 83.5)
- renumbered D2 to D_CHG1, F_USB_2 to F_USB_1, J_VIK_IN_SW_1 to J_L_VIK_1, J_VIK_IN_SW_2 to J_R_VIK_1, R4 to R_B_270, R3 to R_G_330, R_MAT_4 to R_L_A0, R_MAT_14 to R_L_A1, R_MAT_24 to R_L_A2, R_MAT_32 to R_L_RST_1, R_MAT_35 to R_L_SCL_1, R_MAT_34 to R_L_SDA_1, R2 to R_R_470, R_MAT_5 to R_R_A0, R_MAT_16 to R_R_A1, R_MAT_26 to R_R_A2, R_MAT_33 to R_R_RST_1, R_MAT_37 to R_R_SCL_1, R_MAT_36 to R_R_SDA_1, S_MAT_L00 to S_L_00, S_MAT_L01 to S_L_01, S_MAT_L02 to S_L_02, S_MAT_L03 to S_L_03, S_MAT_L04 to S_L_04, S_MAT_L10 to S_L_10, S_MAT_L11 to S_L_11, S_MAT_L12 to S_L_12, S_MAT_L13 to S_L_13, S_MAT_L14 to S_L_14, S_MAT_L15 to S_L_15, S_MAT_L20 to S_L_20, S_MAT_L21 to S_L_21, S_MAT_L22 to S_L_22, S_MAT_L23 to S_L_23, S_MAT_L24 to S_L_24, S_MAT_L25 to S_L_25, S_MAT_L31 to S_L_31, S_MAT_L32 to S_L_32, S_MAT_L33 to S_L_33, S_MAT_L34 to S_L_34, S_MAT_L35 to S_L_35, S_MAT_R00 to S_R_00, S_MAT_R01 to S_R_01, S_MAT_R02 to S_R_02, S_MAT_R03 to S_R_03, S_MAT_R04 to S_R_04, S_MAT_R10 to S_R_10, S_MAT_R11 to S_R_11, S_MAT_R12 to S_R_12, S_MAT_R13 to S_R_13, S_MAT_R14 to S_R_14, S_MAT_R15 to S_R_15, S_MAT_R20 to S_R_20, S_MAT_R21 to S_R_21, S_MAT_R22 to S_R_22, S_MAT_R23 to S_R_23, S_MAT_R24 to S_R_24, S_MAT_R25 to S_R_25, S_MAT_R31 to S_R_31, S_MAT_R32 to S_R_32, S_MAT_R33 to S_R_33, S_MAT_R34 to S_R_34, S_MAT_R35 to S_R_35, U_MAT_2 to U_L_EXT_1, U_MAT_3 to U_R_EXT_1
Connections:
- R_L_A1 pad 1: Net-(U_MAT_2-A1) -> /Left/GND
- R_L_A1 pad 2: /Left/GND -> Net-(U_L_EXT_1-A1)
- R_L_A2 pad 1: Net-(U_MAT_2-A2) -> /Left/GND
- R_L_A2 pad 2: /Left/GND -> Net-(U_L_EXT_1-A2)
- U_L_EXT_1 pad 16: Net-(U_MAT_2-A1) -> Net-(U_L_EXT_1-A1)
- U_L_EXT_1 pad 17: Net-(U_MAT_2-A2) -> Net-(U_L_EXT_1-A2)
Routing:
- net (no net): track 522.4 -> 906.6 mm
- net /Right/CHG_STAT: track 241.1 -> 0.00 mm
- net /Left/SCL: track 201.0 -> 0.00 mm, vias 2 -> 0
- net /Left/SDA: track 194.4 -> 0.00 mm, vias 2 -> 0
- net /Right/C5: track 185.2 -> 1.60 mm
- net /Right/R3: track 232.1 -> 50.9 mm
- net /Left/C5: track 211.3 -> 39.9 mm
- net /Right/R1: track 225.3 -> 61.0 mm
- net /Right/R2: track 223.7 -> 61.0 mm
- net /Right/C4: track 145.0 -> 1.64 mm
- net /Right/C3: track 131.8 -> 1.52 mm
- net /Left/C4: track 168.9 -> 60.4 mm
- net /Right/C2: track 103.0 -> 1.62 mm
- net /Right/R0: track 152.4 -> 51.3 mm
- net /Left/R3: track 233.4 -> 144.2 mm
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