File: pcb/bottom_plate/bottom_plate.kicad_pcb (KiCad board)
At the start: 2 copper layers, 285.8 x 126.1 mm, 33 parts

Commit message: Start redoing bottom plate.
Parts:
- removed JP_CHG_01: Charge_Boost, Jumper:SolderJumper-2_P1.3mm_Open_RoundedPad1.0x1.5mm
- removed J_SWD_01: Conn_01x04, Connector_PinHeader_2.54mm:PinHeader_1x04_P2.54mm_Vertical_SMD_Pin1Left
- removed J_VIK_IN_INTC_01: vik-module-connector, vik:vik-module-connector-horizontal
- removed J_VIK_OUT_DISP_01: VIK_OUT_DISP, vik:vik-keyboard-connector-horizontal
- removed J_VIK_OUT_INTC_01: VIK_OUT_INTC, vik:vik-keyboard-connector-horizontal
- removed J_VIK_OUT_SENS_01, J_VIK_OUT_SENS_02: VIK_OUT_SENS, vik:vik-keyboard-connector-horizontal
- removed J_VIK_OUT_SW_01, J_VIK_OUT_SW_02: VIK_OUT_SW, vik:vik-keyboard-connector-horizontal
- removed Q_EXT_01: AO3401A, Package_TO_SOT_SMD:SOT-23
- removed R_CHG_01: 8K2, Resistor_SMD:R_0201_0603Metric_Pad0.64x0.40mm_HandSolder
- removed R_CHG_02: 2K, Resistor_SMD:R_0201_0603Metric_Pad0.64x0.40mm_HandSolder
- removed R_EXT_01, R_MON_02: 2M, Resistor_SMD:R_0603_1608Metric
- removed R_MON_01: 820K, Resistor_SMD:R_0603_1608Metric
- removed U_CHG_01: MCP73832-2-OT, Package_TO_SOT_SMD:SOT-23-5
- removed U_MCU_01: holyiot-18010-no-underside, mcu:holyiot-18010-no-underside
- added D_POW_1: 1N5819WS, Diode_SMD:D_SOD-323, F.Cu at (227.9, 88.5)
- added FB_USB_1: ~, Inductor_SMD:L_0805_2012Metric, F.Cu at (211.6, 48.5)
- added F_USB_2: SMD0805-050-16V, Fuse:Fuse_0805_2012Metric, F.Cu at (228.0, 54.0)
- added JP_CHG_2: Charge_Boost, Jumper:SolderJumper-2_P1.3mm_Open_RoundedPad1.0x1.5mm, F.Cu at (213.4, 60.1)
- added J_BAT_1: Conn_01x02, Connector_JST:JST_GH_SM02B-GHS-TB_1x02-1MP_P1.25mm_Horizontal, F.Cu at (239.0, 48.1)
- added J_SWD_1: Conn_01x04, Connector_PinHeader_2.54mm:PinHeader_1x04_P2.54mm_Vertical_SMD_Pin1Left, F.Cu at (70.0, 54.0)
- added J_USB_1: USB_C_Receptacle_USB2.0_16P, Connector_USB:USB_C_Receptacle_HRO_TYPE-C-31-M-12, F.Cu at (172.5, 37.5)
- added J_VIK_IN_INTC_2: vik-module-connector, vik:vik-module-connector-horizontal, F.Cu at (188.9, 59.8)
- added J_VIK_OUT_DISP_1: VIK_OUT_DISP, vik:vik-keyboard-connector-horizontal, F.Cu at (98.5, 52.8)
- added J_VIK_OUT_DISP_3: VIK_OUT_DISP, vik:vik-keyboard-connector-horizontal, F.Cu at (189.4, 69.8)
- added J_VIK_OUT_INTC_1: VIK_OUT_INTC, vik:vik-keyboard-connector-horizontal, F.Cu at (109.0, 41.3)
- added J_VIK_OUT_SENS_1: VIK_OUT_SENS, vik:vik-keyboard-connector-horizontal, F.Cu at (126.5, 47.3)
- added J_VIK_OUT_SENS_3: VIK_OUT_SENS, vik:vik-keyboard-connector-horizontal, F.Cu at (189.9, 80.3)
- added J_VIK_OUT_SW_1: VIK_OUT_SW, vik:vik-keyboard-connector-horizontal, F.Cu at (189.5, 93.8)
- added J_VIK_OUT_SW_3: VIK_OUT_SW, vik:vik-keyboard-connector-horizontal, F.Cu at (134.0, 63.3)
- added Q_POW_1: AO3401A, Package_TO_SOT_SMD:SOT-23, F.Cu at (225.6, 80.0)
- added R_CHG_3: 8K2, Resistor_SMD:R_0201_0603Metric_Pad0.64x0.40mm_HandSolder, F.Cu at (162.9, 67.5)
- added R_CHG_4: 2K, Resistor_SMD:R_0201_0603Metric_Pad0.64x0.40mm_HandSolder, F.Cu at (164.1, 70.5)
- added R_MAT_1: 10K, Resistor_SMD:R_0201_0603Metric_Pad0.64x0.40mm_HandSolder, F.Cu at (104.1, 78.0)
- added R_MAT_11: 10K, Resistor_SMD:R_0201_0603Metric_Pad0.64x0.40mm_HandSolder, F.Cu at (104.5, 64.0)
- added R_MAT_12: 10K, Resistor_SMD:R_0201_0603Metric_Pad0.64x0.40mm_HandSolder, F.Cu at (104.1, 73.5)
- added R_MAT_13: 10K, Resistor_SMD:R_0201_0603Metric_Pad0.64x0.40mm_HandSolder, F.Cu at (204.9, 97.2)
- added R_MAT_14: 10K, Resistor_SMD:R_0201_0603Metric_Pad0.64x0.40mm_HandSolder, F.Cu at (204.9, 99.0)
- added R_MAT_2: 10K, Resistor_SMD:R_0201_0603Metric_Pad0.64x0.40mm_HandSolder, F.Cu at (101.1, 81.5)
- added R_MAT_21: 10K, Resistor_SMD:R_0201_0603Metric_Pad0.64x0.40mm_HandSolder, F.Cu at (108.6, 81.5)
- added R_MAT_22: 10K, Resistor_SMD:R_0201_0603Metric_Pad0.64x0.40mm_HandSolder, F.Cu at (111.1, 77.5)
- added R_MAT_23: 10K, Resistor_SMD:R_0201_0603Metric_Pad0.64x0.40mm_HandSolder, F.Cu at (204.9, 100.8)
- added R_MAT_24: 10K, Resistor_SMD:R_0201_0603Metric_Pad0.64x0.40mm_HandSolder, F.Cu at (204.9, 102.5)
- added R_MAT_3: 10K, Resistor_SMD:R_0201_0603Metric_Pad0.64x0.40mm_HandSolder, F.Cu at (204.9, 93.8)
- added R_MAT_31: 10K, Resistor_SMD:R_0201_0603Metric_Pad0.64x0.40mm_HandSolder, F.Cu at (104.0, 68.5)
- added R_MAT_32: 10K, Resistor_SMD:R_0201_0603Metric_Pad0.64x0.40mm_HandSolder, F.Cu at (204.9, 104.2)
- added R_MAT_4: 10K, Resistor_SMD:R_0201_0603Metric_Pad0.64x0.40mm_HandSolder, F.Cu at (204.9, 95.5)
- added R_MON_3: 820K, Resistor_SMD:R_0603_1608Metric, F.Cu at (248.0, 75.0)
- added R_MON_4: 2M, Resistor_SMD:R_0603_1608Metric, F.Cu at (248.0, 71.0)
- added R_POW_1: 100K, Resistor_SMD:R_0201_0603Metric_Pad0.64x0.40mm_HandSolder, F.Cu at (163.6, 84.5)
- added R_USB_1: 5.1K, Resistor_SMD:R_0201_0603Metric_Pad0.64x0.40mm_HandSolder, F.Cu at (164.5, 60.2)
- added R_USB_2: 5.1K, Resistor_SMD:R_0201_0603Metric_Pad0.64x0.40mm_HandSolder, F.Cu at (164.5, 63.0)
- added SW_BAT_1: SW_SPST, library:AS11CH, F.Cu at (225.5, 75.6)
- added SW_RST_1: SW_Push, Button_Switch_SMD:SW_Push_1P1T_NO_E-Switch_TL3301NxxxxxG, F.Cu at (50.5, 53.2)
- added U_CHG_2: MCP73832-2-OT, Package_TO_SOT_SMD:SOT-23-5, F.Cu at (258.4, 69.5)
- added U_MAT_1: MCP23017_SS, Package_SO:SSOP-28_5.3x10.2mm_P0.65mm, F.Cu at (117.5, 62.3)
- added U_MAT_2: MCP23017_SS, Package_SO:SSOP-28_5.3x10.2mm_P0.65mm, F.Cu at (207.0, 84.9)
- added U_MCU_1: holyiot-18010-no-underside, mcu:holyiot-18010-no-underside, F.Cu at (69.7, 27.8)
- added U_POW_1: XC6220B331MR, Package_TO_SOT_SMD:SOT-23-5, F.Cu at (237.9, 81.0)
Connections:
- net /Control_Board/GND renamed /Left/GND
- net /Power_Board/GND renamed /Right/GND
Routing:
- net /Control_Board/5V: track 178.9 -> 0.00 mm
- net /Control_Board/SCLK: track 176.1 -> 0.00 mm
- net /Control_Board/MISO: track 173.8 -> 0.00 mm
- net /Control_Board/VDD: track 159.8 -> 0.00 mm, vias 4 -> 0
- net /Control_Board/VEXT: track 148.0 -> 0.00 mm, vias 2 -> 0
- net /Control_Board/MOSI: track 140.4 -> 0.00 mm, vias 2 -> 0
- net /Control_Board/INT_PMW2: track 136.4 -> 0.00 mm, vias 2 -> 0
- net /Control_Board/SCL: track 128.0 -> 0.00 mm
- net /Control_Board/SDA: track 127.0 -> 0.00 mm
- net /Control_Board/GP22: track 125.3 -> 0.00 mm, vias 2 -> 0
- net /Control_Board/CS_PMW2: track 120.5 -> 0.00 mm, vias 2 -> 0
- net /Control_Board/GP12: track 114.5 -> 0.00 mm, vias 2 -> 0
- net /Control_Board/D-: track 102.3 -> 0.00 mm, vias 2 -> 0
- net /Control_Board/GP31: track 100.6 -> 0.00 mm, vias 2 -> 0
- net /Control_Board/D+: track 100.5 -> 0.00 mm, vias 2 -> 0
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
Commit message: Work on PCBs.
Parts:
- removed FB_USB_1: ~, Inductor_SMD:L_0805_2012Metric
- removed F_USB_2: SMD0805-050-16V, Fuse:Fuse_0805_2012Metric
- removed JP_CHG_2: Charge_Boost, Jumper:SolderJumper-2_P1.3mm_Open_RoundedPad1.0x1.5mm
- removed J_USB_1: USB_C_Receptacle_USB2.0_16P, Connector_USB:USB_C_Receptacle_HRO_TYPE-C-31-M-12
- removed J_VIK_IN_INTC_2: vik-module-connector, vik:vik-module-connector-horizontal
- removed J_VIK_OUT_DISP_3: VIK_OUT_DISP, vik:vik-keyboard-connector-horizontal
- removed J_VIK_OUT_SENS_3: VIK_OUT_SENS, vik:vik-keyboard-connector-horizontal
- removed J_VIK_OUT_SW_3: VIK_OUT_SW, vik:vik-keyboard-connector-horizontal
- removed R_CHG_3: 8K2, Resistor_SMD:R_0201_0603Metric_Pad0.64x0.40mm_HandSolder
- removed R_CHG_4: 2K, Resistor_SMD:R_0201_0603Metric_Pad0.64x0.40mm_HandSolder
- removed R_MAT_1, R_MAT_11, R_MAT_12, R_MAT_13, R_MAT_14, R_MAT_2, R_MAT_21, R_MAT_22, R_MAT_23, R_MAT_24, R_MAT_3, R_MAT_31, R_MAT_32, R_MAT_4: 10K, Resistor_SMD:R_0201_0603Metric_Pad0.64x0.40mm_HandSolder
- removed R_MON_3: 820K, Resistor_SMD:R_0603_1608Metric
- removed R_MON_4: 2M, Resistor_SMD:R_0603_1608Metric
- removed R_USB_1, R_USB_2: 5.1K, Resistor_SMD:R_0201_0603Metric_Pad0.64x0.40mm_HandSolder
- removed U_CHG_2: MCP73832-2-OT, Package_TO_SOT_SMD:SOT-23-5
- removed U_MAT_1, U_MAT_2: MCP23017_SS, Package_SO:SSOP-28_5.3x10.2mm_P0.65mm
- added JP_CHG_1: Charge_Boost, Jumper:SolderJumper-2_P1.3mm_Open_RoundedPad1.0x1.5mm, F.Cu at (186.9, 52.4)
- added J_VIK_IN_INTC_1: vik-module-connector, vik:vik-module-connector-horizontal, F.Cu at (174.6, 94.3)
- added J_VIK_OUT_DISP_2: VIK_OUT_DISP, vik:vik-keyboard-connector-horizontal, F.Cu at (178.6, 57.8)
- added J_VIK_OUT_SENS_2: VIK_OUT_SENS, vik:vik-keyboard-connector-horizontal, F.Cu at (178.6, 66.2)
- added J_VIK_OUT_SW_2: VIK_OUT_SW, vik:vik-keyboard-connector-horizontal, F.Cu at (175.0, 107.8)
- added R_CHG_1: 8K2, Resistor_SMD:R_0201_0603Metric_Pad0.64x0.40mm_HandSolder, F.Cu at (186.2, 55.0)
- added R_CHG_2: 2K, Resistor_SMD:R_0201_0603Metric_Pad0.64x0.40mm_HandSolder, F.Cu at (186.2, 56.8)
- added R_MON_1: 820K, Resistor_SMD:R_0603_1608Metric, F.Cu at (148.0, 58.0)
- added R_MON_2: 2M, Resistor_SMD:R_0603_1608Metric, F.Cu at (148.0, 60.5)
- added U_CHG_1: MCP73832-2-OT, Package_TO_SOT_SMD:SOT-23-5, F.Cu at (187.3, 48.4)
- J_SWD_1: footprint Connector_PinHeader_2.54mm:PinHeader_1x04_P2.54mm_Vertical_SMD_Pin1Left -> Connector_JST:JST_PH_S4B-PH-SM4-TB_1x04-1MP_P2.00mm_Horizontal
- moved J_VIK_OUT_INTC_1 63.4 mm to (143.0, 94.8)
- moved J_VIK_OUT_SW_1 48.4 mm to (143.0, 107.3)
Connections:
- J_VIK_OUT_DISP_1 pad 13: (no net) -> /Left/GND
- J_VIK_OUT_DISP_1 pad 14: (no net) -> /Left/GND
- J_VIK_OUT_DISP_1 pad 6: /Left/VCC -> /Left/VBAT
- J_VIK_OUT_INTC_1 pad 13: (no net) -> /Left/GND
- J_VIK_OUT_INTC_1 pad 14: (no net) -> /Left/GND
- J_VIK_OUT_INTC_1 pad 5: /Left/BATT_MON -> /Left/CHG_STAT
- J_VIK_OUT_INTC_1 pad 6: /Left/VCC -> /Left/VBAT
- J_VIK_OUT_SENS_1 pad 13: (no net) -> /Left/GND
- J_VIK_OUT_SENS_1 pad 14: (no net) -> /Left/GND
- J_VIK_OUT_SENS_1 pad 6: /Left/VCC -> /Left/VBAT
- J_VIK_OUT_SW_1 pad 10: /Left/R1 -> unconnected-(J_VIK_OUT_SW_1-SPI_CS-Pad10)
- J_VIK_OUT_SW_1 pad 11: /Left/R2 -> /Left/MISO
- J_VIK_OUT_SW_1 pad 12: /Left/R3 -> /Left/SCLK
- J_VIK_OUT_SW_1 pad 13: (no net) -> /Left/GND
- J_VIK_OUT_SW_1 pad 14: (no net) -> /Left/GND
- J_VIK_OUT_SW_1 pad 3: /Left/C0 -> /Left/SDA
- J_VIK_OUT_SW_1 pad 4: /Left/C1 -> /Left/SCL
- J_VIK_OUT_SW_1 pad 5: /Left/C2 -> unconnected-(J_VIK_OUT_SW_1-RGB_DO-Pad5)
- J_VIK_OUT_SW_1 pad 6: /Left/C3 -> /Left/VBAT
- J_VIK_OUT_SW_1 pad 7: /Left/C4 -> unconnected-(J_VIK_OUT_SW_1-GP_AD1-Pad7)
- J_VIK_OUT_SW_1 pad 8: /Left/C5 -> /Left/MOSI
- J_VIK_OUT_SW_1 pad 9: /Left/R0 -> unconnected-(J_VIK_OUT_SW_1-GP_AD2-Pad9)
- U_MCU_1 pad 2: /Left/VEXT_EN -> /Left/CHG_STAT
- U_MCU_1 pad 3: /Left/CHG_STAT -> unconnected-(U_MCU_1-[L]_P1.10-Pad3)
- U_MCU_1 pad 35: unconnected-(U_MCU_1-[L]_P1.06-Pad35) -> /Left/CS_DIS1
- U_MCU_1 pad 39: /Left/INT_PMW1 -> unconnected-(U_MCU_1-[L]_P1.02-Pad39)
- U_MCU_1 pad 40: /Left/INT_PMW2 -> unconnected-(U_MCU_1-[L]_P1.01-Pad40)
- U_MCU_1 pad 6: unconnected-(U_MCU_1-[L]_A1_P0.03-Pad6) -> /Left/BATT_MON
- U_MCU_1 pad 7: /Left/BATT_MON -> unconnected-(U_MCU_1-[L]_A0_P0.02-Pad7)

Commit message: Tentatively finish PCBs.
Parts:
- removed SW_BAT_1: SW_SPST, library:AS11CH
- removed SW_RST_1: SW_Push, Button_Switch_SMD:SW_Push_1P1T_NO_E-Switch_TL3301NxxxxxG
- added C1: 4.7uF, Capacitor_SMD:C_1206_3216Metric_Pad1.33x1.80mm_HandSolder, F.Cu at (227.0, 46.0)
- added C2: 4.7uF, Capacitor_SMD:C_1206_3216Metric_Pad1.33x1.80mm_HandSolder, F.Cu at (239.0, 41.0)
- J_SWD_1: footprint Connector_JST:JST_PH_S4B-PH-SM4-TB_1x04-1MP_P2.00mm_Horizontal -> Connector_JST:JST_GH_SM04B-GHS-TB_1x04-1MP_P1.25mm_Horizontal
- R_CHG_1, R_CHG_2, R_POW_1: footprint Resistor_SMD:R_0201_0603Metric_Pad0.64x0.40mm_HandSolder -> Resistor_SMD:R_1206_3216Metric_Pad1.30x1.75mm_HandSolder
- R_MON_1, R_MON_2: footprint Resistor_SMD:R_0603_1608Metric -> Resistor_SMD:R_1206_3216Metric_Pad1.30x1.75mm_HandSolder
- moved J_SWD_1 123.1 mm to (189.8, 82.3), turned to -90 degrees
- moved R_POW_1 74.6 mm to (221.5, 37.5)
- moved U_POW_1 73.3 mm to (177.6, 39.4), turned to 90 degrees
- moved J_VIK_IN_INTC_1 67.0 mm to (240.0, 80.0), turned to 180 degrees
- moved J_VIK_OUT_SW_2 66.2 mm to (240.0, 95.0)
- moved J_VIK_OUT_DISP_2 61.9 mm to (240.0, 50.0)
- moved J_VIK_OUT_DISP_1 61.6 mm to (160.0, 50.0)
- moved J_VIK_OUT_SENS_2 61.4 mm to (240.0, 65.0)
- moved D_POW_1 50.5 mm to (226.0, 38.0), turned to 180 degrees
- moved J_BAT_1 45.7 mm to (209.5, 83.0), turned to 90 degrees
- moved R_MON_2 45.2 mm to (188.5, 40.5)
- moved H5 42.0 mm to (104.2, 98.0)
- moved H1 42.0 mm to (98.1, 18.1)
- moved H10 42.0 mm to (204.0, 78.2)
- moved H12 42.0 mm to (223.9, 134.0)
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Connections:
- J_BAT_1 pad 1: Net-(J_BAT_1-Pin_1) -> /Right/VBAT
- J_BAT_1 pad MP: (no net) -> /Right/GND
- J_SWD_1 pad MP: (no net) -> /Left/GND
- J_VIK_IN_INTC_1 pad 7: /Right/VBAT -> /Right/VCC
- J_VIK_IN_INTC_1 pad 8: /Right/CHG_STAT -> /Right/CS_DIS2
- J_VIK_OUT_DISP_1 pad 6: /Left/VBAT -> /Left/VCC
- J_VIK_OUT_DISP_2 pad 6: /Right/VBAT -> /Right/VCC
- J_VIK_OUT_INTC_1 pad 5: /Left/CHG_STAT -> /Left/CS_DIS2
- J_VIK_OUT_INTC_1 pad 6: /Left/VBAT -> /Left/VCC
- J_VIK_OUT_SENS_1 pad 6: /Left/VBAT -> /Left/VCC
- J_VIK_OUT_SENS_2 pad 6: /Right/VBAT -> /Right/VCC
- J_VIK_OUT_SW_1 pad 6: /Left/VBAT -> /Left/VCC
- J_VIK_OUT_SW_1 pad 7: unconnected-(J_VIK_OUT_SW_1-GP_AD1-Pad7) -> /Left/RST
- J_VIK_OUT_SW_2 pad 5: unconnected-(J_VIK_OUT_SW_2-RGB_DO-Pad5) -> /Right/CHG_STAT
- R_MON_1 pad 1: /Left/VBAT -> /Left/VCC
- U_MCU_1 pad 2: /Left/CHG_STAT -> unconnected-(U_MCU_1-[L]_P1.11-Pad2)
- U_MCU_1 pad 36: unconnected-(U_MCU_1-[L]_P1.04-Pad36) -> /Left/CS_DIS2
- U_MCU_1 pad 48: Net-(U_MCU_1-Reset/P0.18) -> /Left/RST
- U_POW_1 pad 1: /Right/VCC -> /Left/VCC
- U_POW_1 pad 2: /Right/GND -> /Left/GND
- U_POW_1 pad 3: /Right/VCC -> /Left/VCC
- U_POW_1 pad 5: /Right/VDD -> /Left/VDD
Routing:
- net /Left/VDD: track 0.00 -> 177.7 mm, vias 0 -> 2
- net /Left/VCC: track 0.00 -> 126.6 mm, vias 0 -> 2
- net /Left/SCLK: track 0.00 -> 108.3 mm, vias 0 -> 2
- net /Left/MISO: track 0.00 -> 105.9 mm, vias 0 -> 2
- net /Left/MOSI: track 0.00 -> 104.9 mm, vias 0 -> 2
- net /Right/VUSB: track 0.00 -> 99.5 mm
- net /Left/SWD: track 0.00 -> 96.7 mm, vias 0 -> 2
- net /Left/SWC: track 0.00 -> 95.2 mm, vias 0 -> 2
- net /Left/BATT_MON: track 0.00 -> 93.0 mm, vias 0 -> 2
- net /Left/SCL: track 0.00 -> 92.0 mm
- net /Left/SDA: track 0.00 -> 91.0 mm
- net /Left/RST: track 0.00 -> 76.0 mm, vias 0 -> 2
- net /Left/CS_PMW2: track 0.00 -> 72.4 mm, vias 0 -> 2
- net /Right/CHG_STAT: track 0.00 -> 71.9 mm
- net /Left/CS_DIS2: track 0.00 -> 70.0 mm, vias 0 -> 2
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
Commit message: Add ESD protection to PCBs.
Parts:
- added U_ESD_D1: CM1293A, Package_TO_SOT_SMD:SOT-23-6, F.Cu at (156.0, 103.5)
- added U_ESD_D2: CM1293A, Package_TO_SOT_SMD:SOT-23-6, F.Cu at (164.0, 103.5)
- added U_ESD_D3: CM1293A, Package_TO_SOT_SMD:SOT-23-6, F.Cu at (153.5, 84.5)
- added U_ESD_D4: CM1293A, Package_TO_SOT_SMD:SOT-23-6, F.Cu at (236.0, 103.5)
- added U_ESD_D5: CM1293A, Package_TO_SOT_SMD:SOT-23-6, F.Cu at (244.1, 103.5)
Routing:
- net /Right/CS_PMW2: track 19.1 -> 65.7 mm, vias 0 -> 2
- net /Left/GND: track 63.5 -> 98.1 mm, vias 9 -> 10
- net /Left/CS_DIS2: track 70.0 -> 103.3 mm, vias 2 -> 3
- net /Left/CS_PMW2: track 72.4 -> 104.1 mm, vias 2 -> 3
- net /Right/CS_DIS2: track 37.3 -> 63.4 mm, vias 2 -> 3
- net /Left/VDD: track 177.7 -> 202.8 mm
- net /Right/VDD: track 45.0 -> 69.8 mm
- net /Right/VUSB: track 99.5 -> 82.5 mm, vias 0 -> 2
- net /Right/SCLK: track 45.0 -> 58.1 mm
- net /Left/SCLK: track 108.3 -> 121.4 mm
- net /Right/CHG_STAT: track 71.9 -> 59.2 mm, vias 0 -> 2
- net /Left/D+: track 65.5 -> 77.6 mm, vias 2 -> 3
- net /Left/SDA: track 91.0 -> 101.9 mm
- net /Right/SDA: track 45.0 -> 55.7 mm
- net /Right/MISO: track 45.0 -> 55.5 mm
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