File: pcb/bottom_plate/bottom_plate.kicad_pcb (KiCad board)
At the start: 2 copper layers, 285.8 x 126.1 mm, 44 parts

Commit message: Rework PCBs to ensure adequate clearance between them.
Parts:
- H1, H10, H11, H12, H2, H3, H4, H5, H6, H7, H8, H9: footprint MountingHole:MountingHole_2.2mm_M2_Pad -> MountingHole:MountingHole_2.2mm_M2
- moved R_MON_2 113.8 mm to (75.5, 27.1), turned to 90 degrees
- moved R_MON_1 108.3 mm to (75.5, 32.1), turned to 90 degrees
- moved U_ESD_D2 93.2 mm to (86.5, 51.7), turned to 180 degrees
- moved U_ESD_D1 89.7 mm to (86.5, 46.8), turned to 0 degrees
- moved U_POW_1 89.4 mm to (88.2, 42.6), turned to 180 degrees
- moved U_ESD_D5 58.9 mm to (220.6, 49.5), turned to 0 degrees
- moved R_POW_1 55.7 mm to (240.0, 90.0), turned to -90 degrees
- moved C2 49.0 mm to (237.5, 90.0), turned to -90 degrees
- moved Q_POW_1 44.9 mm to (237.0, 84.5), turned to 90 degrees
- moved U_ESD_D4 44.8 mm to (220.6, 61.5), turned to 0 degrees
- moved C1 44.7 mm to (235.0, 90.0)
- moved D_POW_1 43.3 mm to (238.5, 79.5)
- moved U_CHG_1 40.8 mm to (234.0, 79.5), turned to 0 degrees
- moved JP_CHG_1 39.9 mm to (237.5, 74.2), turned to 90 degrees
- moved R_CHG_1 34.8 mm to (234.0, 73.3), turned to 90 degrees
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Connections:
- U_ESD_D1 pad 1: /Left/CS_DIS2 -> /Left/CS_PMW2
- U_ESD_D1 pad 3: /Left/CS_PMW2 -> /Left/CS_DIS2
- U_ESD_D1 pad 4: /Left/SCL -> /Left/SDA
- U_ESD_D1 pad 6: /Left/SDA -> /Left/SCL
- U_ESD_D2 pad 3: /Left/SCLK -> /Left/MOSI
- U_ESD_D2 pad 6: /Left/MOSI -> /Left/SCLK
Routing:
- net /Left/RST: track 77.1 -> 164.8 mm, vias 2 -> 0
- net /Left/BATT_MON: track 93.0 -> 5.73 mm, vias 2 -> 0
- net /Left/VCC: track 134.4 -> 213.2 mm, vias 4 -> 6
- net /Left/SWC: track 95.2 -> 160.9 mm, vias 2 -> 0
- net /Left/SWD: track 96.7 -> 157.5 mm, vias 2 -> 0
- net /Left/SCLK: track 121.4 -> 181.1 mm, vias 2 -> 4
- net /Left/MISO: track 116.4 -> 175.8 mm, vias 2 -> 4
- net /Right/VUSB: track 82.5 -> 26.8 mm, vias 2 -> 0
- net /Right/CHG_STAT: track 59.2 -> 8.65 mm, vias 2 -> 0
- net /Left/SCL: track 102.3 -> 151.1 mm, vias 0 -> 6
- net /Left/MOSI: track 115.3 -> 161.2 mm, vias 2 -> 6
- net /Left/CS_DIS1: track 54.1 -> 97.7 mm, vias 2 -> 0
- net /Left/SDA: track 101.9 -> 145.1 mm, vias 0 -> 6
- net /Right/CS_PMW2: track 65.7 -> 27.3 mm, vias 2 -> 0
- net /Left/D-: track 74.5 -> 112.0 mm, vias 3 -> 0
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