File: pcb/bottom_plate/left.kicad_sch (KiCad schematic)
At the start: 14 parts

Commit message: Start redoing bottom plate.
Parts:
- removed Q_EXT_1: AO3401A, Package_TO_SOT_SMD:SOT-23, symbol Transistor_FET:AO3401A
- removed R_EXT_1: 2M, Resistor_SMD:R_0603_1608Metric, symbol Device:R
- added R_MAT_13, R_MAT_14, R_MAT_23, R_MAT_24, R_MAT_3, R_MAT_32, R_MAT_4: 10K, Resistor_SMD:R_0201_0603Metric_Pad0.64x0.40mm_HandSolder, symbol Device:R
- added SW_RST_1: SW_Push, Button_Switch_SMD:SW_Push_1P1T_NO_E-Switch_TL3301NxxxxxG, symbol Switch:SW_Push
- added U_MAT_2: MCP23017_SS, Package_SO:SSOP-28_5.3x10.2mm_P0.65mm, symbol Interface_Expansion:MCP23017x-x-SS
Connections:
- net BATT_MON: now also J_VIK_OUT_INTC_1.5 (RGB_DO)
- net CS_DIS1: now also U_MAT_2.25 (GPA4); no longer U_MCU_1.35 ([L]_P1.06)
- net D+: now also J_VIK_OUT_INTC_1.7 (GP_AD1); no longer J_VIK_OUT_SW_1.9 (GP_AD2)
- net D-: now also J_VIK_OUT_INTC_1.9 (GP_AD2); no longer J_VIK_OUT_SW_1.7 (GP_AD1)
- net GND: now also R_MAT_14.2, R_MAT_24.2, R_MAT_4.2, SW_RST_1.1, U_MAT_2.10 (V_{SS})
- net INT_PMW2: no longer J_VIK_OUT_INTC_1.7 (GP_AD1)
- net MISO: no longer J_VIK_OUT_SW_1.11 (MISO)
- net MOSI: no longer J_VIK_OUT_SW_1.8 (MOSI)
- net SCL: now also U_MAT_2.13 (SDA); no longer J_VIK_OUT_SW_1.4 (SCL)
- net SCLK: no longer J_VIK_OUT_SW_1.12 (SCLK)
- net SDA: now also U_MAT_2.12 (SCK); no longer J_VIK_OUT_SW_1.3 (SDA)
- net VDD: now also R_MAT_13.1, R_MAT_23.1, R_MAT_3.1, R_MAT_32.1, U_MAT_2.9 (V_{DD})
- net 5V renamed VCC
- net VCC: no longer J_VIK_OUT_SW_1.6 (5V)
- net CS_SW1: no longer names the net of U_MCU_1.36 ([L]_P1.04)
- net GP12: no longer names the net of J_VIK_OUT_SENS_1.9 (GP_AD2)
- net GP12: no longer U_MCU_1.8 ([L]_A4_P0.28)
- net GP22: no longer names the net of U_MCU_1.9 ([L]_A5_P0.29)
- net GP22: no longer J_VIK_OUT_INTC_1.9 (GP_AD2)
- net GP31: no longer names the net of J_VIK_OUT_DISP_1.7 (GP_AD1)
- net GP31: no longer U_MCU_1.10 ([L]_A6_P0.30)
- net GP32: no longer names the net of J_VIK_OUT_DISP_1.9 (GP_AD2)
- net GP32: no longer U_MCU_1.11 ([L]_A7_P0.31)
- net RST: no longer names the net of U_MCU_1.48 (Reset/P0.18)
- net RST: now also SW_RST_1.2; no longer J_VIK_OUT_SW_1.10 (SPI_CS)
- removed net VEXT: J_VIK_OUT_DISP_1.5 (RGB_DO), J_VIK_OUT_INTC_1.5 (RGB_DO), J_VIK_OUT_SENS_1.5 (RGB_DO), J_VIK_OUT_SW_1.5 (RGB_DO)
- new net: R_MAT_3.2, R_MAT_4.1, U_MAT_2.15 (A0)
- new net: R_MAT_23.2, R_MAT_24.1, U_MAT_2.17 (A2)
- new net: R_MAT_13.2, R_MAT_14.1, U_MAT_2.16 (A1)
- new net: R_MAT_32.2, U_MAT_2.18 (~{RESET})
- new net C0: J_VIK_OUT_SW_1.3 (SDA), U_MAT_2.1 (GPB0)
- new net C1: J_VIK_OUT_SW_1.4 (SCL), U_MAT_2.2 (GPB1)
- new net C2: J_VIK_OUT_SW_1.5 (RGB_DO), U_MAT_2.3 (GPB2)
- new net C3: J_VIK_OUT_SW_1.6 (5V), U_MAT_2.4 (GPB3)
- new net C4: J_VIK_OUT_SW_1.7 (GP_AD1), U_MAT_2.5 (GPB4)
- new net C5: J_VIK_OUT_SW_1.8 (MOSI), U_MAT_2.6 (GPB5)
- new net R0: J_VIK_OUT_SW_1.9 (GP_AD2), U_MAT_2.21 (GPA0)
- new net R1: J_VIK_OUT_SW_1.10 (SPI_CS), U_MAT_2.22 (GPA1)
- new net R2: J_VIK_OUT_SW_1.11 (MISO), U_MAT_2.23 (GPA2)
- new net R3: J_VIK_OUT_SW_1.12 (SCLK), U_MAT_2.24 (GPA3)
- no-connect marks 9 -> 27
Other:
- note removed: "External Power"
- moved on the sheet: H1, H2, H3, H4, H5, H6, J_SWD_1, J_VIK_OUT_DISP_1, J_VIK_OUT_INTC_1, J_VIK_OUT_SENS_1, J_VIK_OUT_SW_1

Commit message: Work on PCBs.
Parts:
- removed R_MAT_13, R_MAT_14, R_MAT_23, R_MAT_24, R_MAT_3, R_MAT_32, R_MAT_4: 10K, Resistor_SMD:R_0201_0603Metric_Pad0.64x0.40mm_HandSolder, symbol Device:R
- removed U_MAT_2: MCP23017_SS, Package_SO:SSOP-28_5.3x10.2mm_P0.65mm, symbol Interface_Expansion:MCP23017x-x-SS
- added R_MON_1: 820K, Resistor_SMD:R_0603_1608Metric, symbol Device:R
- added R_MON_2: 2M, Resistor_SMD:R_0603_1608Metric, symbol Device:R
- added U_POW_1: XC6220B331MR, Package_TO_SOT_SMD:SOT-23-5, symbol Regulator_Linear:XC6220B331MR
- J_SWD_1: footprint Connector_PinHeader_2.54mm:PinHeader_1x04_P2.54mm_Vertical_SMD_Pin1Left -> Connector_JST:JST_GH_SM04B-GHS-TB_1x04-1MP_P1.25mm_Horizontal
Connections:
- net C0 is gone; now on net SDA: J_VIK_OUT_SW_1.3 (SDA)
- net C1 is gone; now on net SCL: J_VIK_OUT_SW_1.4 (SCL)
- net C3 is gone; now on net VCC: J_VIK_OUT_SW_1.6 (5V)
- net C5 is gone; now on net MOSI: J_VIK_OUT_SW_1.8 (MOSI)
- net R2 is gone; now on net MISO: J_VIK_OUT_SW_1.11 (MISO)
- net R3 is gone; now on net SCLK: J_VIK_OUT_SW_1.12 (SCLK)
- net VEXT_EN is gone; now on net CHG_STAT: U_MCU_1.2 ([L]_P1.11)
- net BATT_MON: now also U_MCU_1.6 ([L]_A1_P0.03), R_MON_1.2, R_MON_2.1; no longer J_VIK_OUT_INTC_1.5 (RGB_DO), U_MCU_1.7 ([L]_A0_P0.02)
- net CHG_STAT: now also J_VIK_OUT_INTC_1.5 (RGB_DO); no longer U_MCU_1.3 ([L]_P1.10)
- net CS_DIS1: now also U_MCU_1.35 ([L]_P1.06)
- net GND: now also J_VIK_OUT_DISP_1.13 (MP), J_VIK_OUT_DISP_1.14 (MP), J_VIK_OUT_INTC_1.13 (MP), J_VIK_OUT_INTC_1.14 (MP), J_VIK_OUT_SENS_1.13 (MP), J_VIK_OUT_SENS_1.14 (MP), J_VIK_OUT_SW_1.13 (MP), J_VIK_OUT_SW_1.14 (MP), R_MON_2.2, U_POW_1.2 (GND)
- net INT_PMW1: no longer U_MCU_1.39 ([L]_P1.02)
- net VCC: now also R_MON_1.1, U_POW_1.1 (VIN), U_POW_1.3 (CE)
- net VDD: now also U_POW_1.5 (VOUT)
- net C2: no longer names the net of J_VIK_OUT_SW_1.5 (RGB_DO)
- net C4: no longer names the net of J_VIK_OUT_SW_1.7 (GP_AD1)
- net INT_PMW2: no longer names the net of U_MCU_1.40 ([L]_P1.01)
- net R0: no longer names the net of J_VIK_OUT_SW_1.9 (GP_AD2)
- net R1: no longer names the net of J_VIK_OUT_SW_1.10 (SPI_CS)
- no-connect marks 27 -> 26
Other:
- note added: "Battery Monitor"
- moved on the sheet: J_SWD_1

Commit message: Tentatively finish PCBs.
Parts:
- removed SW_RST_1: SW_Push, Button_Switch_SMD:SW_Push_1P1T_NO_E-Switch_TL3301NxxxxxG, symbol Switch:SW_Push
- J_SWD_1: symbol Connector_Generic:Conn_01x04 -> Connector_Generic_MountingPin:Conn_01x04_MountingPin
- R_MON_1, R_MON_2: footprint Resistor_SMD:R_0603_1608Metric -> Resistor_SMD:R_1206_3216Metric_Pad1.30x1.75mm_HandSolder
Connections:
- net GND: now also J_SWD_1.MP (MountPin)
- net RST: now reaches U_MCU_1.48 (Reset/P0.18)
- net RST: now also J_VIK_OUT_SW_1.7 (GP_AD1)
- net CS_DIS2: now reaches U_MCU_1.36 ([L]_P1.04)
- net CS_DIS2: now also J_VIK_OUT_INTC_1.5 (RGB_DO)
- net CHG_STAT: no longer names the net of U_MCU_1.2 ([L]_P1.11)
- net CHG_STAT: no longer J_VIK_OUT_INTC_1.5 (RGB_DO)
- no-connect marks 26 -> 25
Changed lines of the file:
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@@
+	)
+	(no_connect
+		(at 39.37 43.18)
 	)
 	(no_connect
@@
 	)
 	(no_connect
-		(at 77.47 50.8)
-	)
-	(no_connect
 		(at 39.37 58.42)
 	)
@@
 	(no_connect
 		(at 77.47 60.96)
-	)
-	(no_connect
-		(at 171.45 106.68)
 	)
 	(no_connect
@@
 	(wire
 		(pts
-			(xy 63.5 92.71) (xy 63.5 87.63)
+			(xy 238.76 53.34) (xy 245.11 53.34)
 		)
 		(stroke
@@
 		)
 	)
-	(wire
+	(polyline
 		(pts
-			(xy 238.76 53.34) (xy 245.11 53.34)
+			(xy 252.73 91.44) (xy 241.3 88.9)
 		)
 		(stroke
@@
 		)
 	)
-	(polyline
+	(wire
 		(pts
-			(xy 252.73 91.44) (xy 241.3 88.9)
+			(xy 245.11 50.8) (xy 245.11 53.34)
 		)
 		(stroke
@@
 	(wire
 		(pts
-			(xy 245.11 50.8) (xy 245.11 53.34)
+			(xy 245.11 53.34) (xy 245.11 55.88)
 		)
 		(stroke
@@
 	(wire
 		(pts
-			(xy 245.11 53.34) (xy 245.11 55.88)
+			(xy 245.11 63.5) (xy 245.11 66.04)
 		)
 		(stroke
@@
 		)
 	)
-	(wire
-		(pts
-			(xy 245.11 63.5) (xy 245.11 66.04)
-		)
-		(stroke
-			(width 0)
-			(type default)
-		)
-	)
 	(label "GND"
 		(at 129.54 147.32 180)
@@
 		)
 	)
+	(label "RST"
+		(at 171.45 106.68 180)
+		(effects
+			(font
+				(size 1.524 1.524)
+			)
+			(justify right bottom)
+		)
+	)
 	(label "CS_DIS1"
 		(at 125.73 114.3 180)
@@
 		)
 	)
+	(label "RST"
+		(at 63.5 87.63 270)
+		(effects
+			(font
+				(size 1.524 1.524)
+			)
+			(justify right bottom)
+		)
+	)
 	(label "VCC"
 		(at 228.6 91.44 180)
@@
 		)
 	)
+	(label "GND"
+		(at 134.62 154.94 270)
+		(effects
+			(font
+				(size 1.524 1.524)
+			)
+			(justify right bottom)
+		)
+	)
 	(label "SCLK"
 		(at 171.45 62.23 180)
@@
 		)
 	)
-	(label "CHG_STAT"
+	(label "CS_DIS2"
 		(at 125.73 44.45 180)
-		(effects
-			(font
-				(size 1.524 1.524)
-			)
-			(justify right bottom)
-		)
-	)
-	(label "CHG_STAT"
-		(at 39.37 43.18 180)
-		(effects
-			(font
-				(size 1.524 1.524)
-			)
-			(justify right bottom)
-		)
-	)
-	(label "GND"
-		(at 63.5 102.87 270)
 		(effects
 			(font
@@
 			)
 			(justify right bottom)
+		)
+	)
+	(label "CS_DIS2"
+		(at 77.47 50.8 0)
+		(effects
+			(font
+				(size 1.524 1.524)
+			)
+			(justify left bottom)
 		)
 	)
@@
 	)
 	(symbol
-		(lib_id "Switch:SW_Push")
-		(at 63.5 97.79 90)
-		(unit 1)
-		(body_style 1)
-		(exclude_from_sim no)
-		(in_bom yes)
-		(on_board yes)
-		(in_pos_files yes)
-		(dnp no)
-		(fields_autoplaced yes)
-		(property "Reference" "SW_RST_1"
-			(at 64.77 96.5199 90)
-			(show_name no)
-			(do_not_autoplace no)
-			(effects
-				(font
-					(size 1.27 1.27)
-				)
-				(justify right)
-			)
-		)
-		(property "Value" "SW_Push"
-			(at 64.77 99.0599 90)
-			(show_name no)
-			(do_not_autoplace no)
-			(effects
-				(font
-					(size 1.27 1.27)
-				)
-				(justify right)
-			)
-		)
-		(property "Footprint" "Button_Switch_SMD:SW_Push_1P1T_NO_E-Switch_TL3301NxxxxxG"
-			(at 58.42 97.79 0)
-			(hide yes)
-			(show_name no)
-			(do_not_autoplace no)
-			(effects
-				(font
-					(size 1.27 1.27)
-				)
-			)
-		)
-		(property "Datasheet" ""
-			(at 58.42 97.79 0)
-			(hide yes)
-			(show_name no)
-			(do_not_autoplace no)
-			(effects
-				(font
-					(size 1.27 1.27)
-				)
-			)
-		)
-		(property "Description" "Push button switch, generic, two pins"
-			(at 63.5 97.79 0)
-			(hide yes)
-			(show_name no)
-			(do_not_autoplace no)
-			(effects
-				(font
-					(size 1.27 1.27)
-				)
-			)
-		)
-		(pin "1"
-		)
-		(pin "2"
-		)
-		(instances
-			(project "bottom_plate"
-				(path "/b41c5c8d-a6b2-4633-9a6f-a9fc0b4f40ca/ebd9436f-55ad-414e-b8cc-8a07a71cfe92"
-					(reference "SW_RST_1")
-					(unit 1)
-				)
-			)
-		)
-	)
-	(symbol
 		(lib_id "Mechanical:MountingHole_Pad")
 		(at 50.8 204.47 0)
@@
 			)
 		)
-		(property "Footprint" "Resistor_SMD:R_0603_1608Metric"
+		(property "Footprint" "Resistor_SMD:R_1206_3216Metric_Pad1.30x1.75mm_HandSolder"
 			(at 243.332 46.99 90)
 			(hide yes)
@@
 			(effects
 				(font
-					(face "Standard Symbols PS")
 					(size 1.27 1.27)
 				)
@@
 			)
 		)
-		(property "Footprint" "Resistor_SMD:R_0603_1608Metric"
+		(property "Footprint" "Resistor_SMD:R_1206_3216Metric_Pad1.30x1.75mm_HandSolder"
 			(at 243.332 59.69 90)
 			(hide yes)
@@
 	)
 	(symbol
-		(lib_id "Connector_Generic:Conn_01x04")
+		(lib_id "Connector_Generic_MountingPin:Conn_01x04_MountingPin")
 		(at 134.62 144.78 0)
 		(unit 1)
@@
 		(fields_autoplaced yes)
 		(property "Reference" "J_SWD_1"
-			(at 137.16 144.7799 0)
+			(at 137.16 145.1355 0)
 			(show_name no)
 			(do_not_autoplace no)
@@
 		)
 		(property "Value" "Conn_01x04"
-			(at 137.16 147.3199 0)
+			(at 137.16 147.6755 0)
 			(show_name no)
 			(do_not_autoplace no)
@@
 			)
 		)
-		(property "Description" "Generic connector, single row, 01x04, script generated (kicad-library-utils/schlib/autogen/connector/)"
+		(property "Description" "Generic connectable mounting pin connector, single row, 01x04, script generated (kicad-library-utils/schlib/autogen/connector/)"
 			(at 134.62 144.78 0)
 			(hide yes)
@@
 		(pin "4"
 		)
+		(pin "MP"
+		)
 		(instances

Commit message: Add ESD protection to PCBs.
Parts:
- added U_ESD_D1, U_ESD_D2, U_ESD_D3: CM1293A, Package_TO_SOT_SMD:SOT-23-6, symbol Power_Protection:SRV05-4
Connections:
- net CS_DIS2: now also U_ESD_D1.1 (IO1)
- net CS_PMW2: now also U_ESD_D1.3 (IO2)
- net D+: now also U_ESD_D3.4 (IO3)
- net D-: now also U_ESD_D3.6 (IO4)
- net GND: now also U_ESD_D1.2 (VN), U_ESD_D2.2 (VN), U_ESD_D3.2 (VN)
- net MISO: now also U_ESD_D2.4 (IO3)
- net MOSI: now also U_ESD_D2.6 (IO4)
- net SCL: now also U_ESD_D1.4 (IO3)
- net SCLK: now also U_ESD_D2.3 (IO2)
- net SDA: now also U_ESD_D1.6 (IO4)
- net VCC: now also U_ESD_D3.5 (VP)
- net VDD: now also U_ESD_D1.5 (VP), U_ESD_D2.5 (VP)
- no-connect marks 25 -> 28
