File: pcb/bottom_plate/right.kicad_sch (KiCad schematic)
At the start: 16 parts

Commit message: Start redoing bottom plate.
Parts:
- added D_POW_1: 1N5819WS, Diode_SMD:D_SOD-323, symbol Diode:1N5819WS
- added FB_USB_1: (no value), Inductor_SMD:L_0805_2012Metric, symbol Device:FerriteBead
- added F_USB_2: SMD0805-050-16V, Fuse:Fuse_0805_2012Metric, symbol Device:Fuse
- added J_BAT_1: Conn_01x02, Connector_JST:JST_GH_SM02B-GHS-TB_1x02-1MP_P1.25mm_Horizontal, symbol Connector_Generic:Conn_01x02
- added J_USB_1: USB_C_Receptacle_USB2.0_16P, Connector_USB:USB_C_Receptacle_HRO_TYPE-C-31-M-12, symbol Connector:USB_C_Receptacle_USB2.0_16P
- added Q_POW_1: AO3401A, Package_TO_SOT_SMD:SOT-23, symbol Transistor_FET:AO3401A
- added R_MAT_1, R_MAT_11, R_MAT_12, R_MAT_2, R_MAT_21, R_MAT_22, R_MAT_31: 10K, Resistor_SMD:R_0201_0603Metric_Pad0.64x0.40mm_HandSolder, symbol Device:R
- added R_POW_1: 100K, Resistor_SMD:R_0201_0603Metric_Pad0.64x0.40mm_HandSolder, symbol Device:R
- added R_USB_1, R_USB_2: 5.1K, Resistor_SMD:R_0201_0603Metric_Pad0.64x0.40mm_HandSolder, symbol Device:R
- added SW_BAT_1: SW_SPST, library:AS11CH, symbol Switch:SW_SPST
- added U_MAT_1: MCP23017_SS, Package_SO:SSOP-28_5.3x10.2mm_P0.65mm, symbol Interface_Expansion:MCP23017x-x-SS
- added U_POW_1: XC6220B331MR, Package_TO_SOT_SMD:SOT-23-5, symbol Regulator_Linear:XC6220B331MR
- J_VIK_OUT_DISP_3: now fitted; now in the parts list
- renumbered H16 to H10, H17 to H11, H18 to H12, H13 to H7, H14 to H8, H15 to H9
Connections:
- net 5V: no longer J_VIK_IN_INTC_2.7 (5V), J_VIK_OUT_SENS_3.6 (5V), J_VIK_OUT_SW_3.6 (5V)
- net BATT_MON: now also J_VIK_IN_INTC_2.8 (RGB_DO); no longer J_VIK_IN_INTC_2.4 (GP_AD2)
- net GND: now also FB_USB_1.2, J_BAT_1.2 (Pin_2), J_USB_1.A1 (GND), J_USB_1.A12 (GND), J_USB_1.B1 (GND), J_USB_1.B12 (GND), R_MAT_1.2, R_MAT_11.2, R_MAT_21.2, R_POW_1.2, R_USB_1.2, R_USB_2.2, U_MAT_1.10 (V_{SS}), U_POW_1.2 (GND)
- net INT_PMW2: no longer J_VIK_IN_INTC_2.6 (GP_AD1)
- net MISO: no longer J_VIK_OUT_SW_3.11 (MISO)
- net MOSI: no longer J_VIK_OUT_SW_3.8 (MOSI)
- net SCL: now also U_MAT_1.13 (SDA); no longer J_VIK_OUT_SW_3.4 (SCL)
- net SCLK: no longer J_VIK_OUT_SW_3.12 (SCLK)
- net SDA: now also U_MAT_1.12 (SCK); no longer J_VIK_OUT_SW_3.3 (SDA)
- net VBAT: now also Q_POW_1.3 (D), SW_BAT_1.1 (A)
- net VDD: now also R_MAT_12.1, R_MAT_2.1, R_MAT_22.1, R_MAT_31.1, U_MAT_1.9 (V_{DD}), U_POW_1.5 (VOUT)
- net R1: now reaches J_VIK_OUT_SW_3.10 (SPI_CS)
- net R1: now also U_MAT_1.22 (GPA1)
- net C4: now reaches J_VIK_OUT_SW_3.7 (GP_AD1)
- net C4: now also U_MAT_1.5 (GPB4)
- net R0: now reaches J_VIK_OUT_SW_3.9 (GP_AD2)
- net R0: now also U_MAT_1.21 (GPA0)
- net CS_DIS1 renamed CS_DIS2
- net CS_DIS2: now also U_MAT_1.25 (GPA4)
- net GP31: no longer names the net of J_VIK_OUT_DISP_3.7 (GP_AD1)
- net GP32: no longer names the net of J_VIK_OUT_DISP_3.9 (GP_AD2)
- removed net VEXT: J_VIK_IN_INTC_2.8 (RGB_DO), J_VIK_OUT_DISP_3.5 (RGB_DO), J_VIK_OUT_SENS_3.5 (RGB_DO), J_VIK_OUT_SW_3.5 (RGB_DO)
- new net: R_MAT_11.1, R_MAT_12.2, U_MAT_1.16 (A1)
- new net: J_BAT_1.1 (Pin_1), SW_BAT_1.2 (B)
- new net: R_MAT_1.1, R_MAT_2.2, U_MAT_1.15 (A0)
- new net: R_MAT_21.1, R_MAT_22.2, U_MAT_1.17 (A2)
- new net: R_MAT_31.2, U_MAT_1.18 (~{RESET})
- new net: J_USB_1.A5 (CC1), R_USB_1.1
- new net: J_USB_1.B5 (CC2), R_USB_2.1
- new net C0: J_VIK_OUT_SW_3.3 (SDA), U_MAT_1.1 (GPB0)
- new net C1: J_VIK_OUT_SW_3.4 (SCL), U_MAT_1.2 (GPB1)
- new net C2: J_VIK_OUT_SW_3.5 (RGB_DO), U_MAT_1.3 (GPB2)
- new net C3: J_VIK_OUT_SW_3.6 (5V), U_MAT_1.4 (GPB3)
- new net C5: J_VIK_OUT_SW_3.8 (MOSI), U_MAT_1.6 (GPB5)
- new net D+: J_USB_1.A6 (D+), J_USB_1.B6 (D+), J_VIK_IN_INTC_2.6 (GP_AD1)
- new net D-: J_USB_1.A7 (D-), J_USB_1.B7 (D-), J_VIK_IN_INTC_2.4 (GP_AD2)
- new net R2: J_VIK_OUT_SW_3.11 (MISO), U_MAT_1.23 (GPA2)
- new net R3: J_VIK_OUT_SW_3.12 (SCLK), U_MAT_1.24 (GPA3)
- new net SH: FB_USB_1.1, J_USB_1.SH (SHIELD)
- new net VCC: D_POW_1.1 (K), J_VIK_IN_INTC_2.7 (5V), J_VIK_OUT_SENS_3.6 (5V), Q_POW_1.2 (S), U_POW_1.1 (VIN), U_POW_1.3 (CE)
- new net VUSB: D_POW_1.2 (A), F_USB_2.2, Q_POW_1.1 (G), R_POW_1.1
- new net VUSB_RAW: F_USB_2.1, J_USB_1.A4 (VBUS), J_USB_1.A9 (VBUS), J_USB_1.B4 (VBUS), J_USB_1.B9 (VBUS)
- no-connect marks 4 -> 14
Other:
- note added: "Port"
- note added: "VBUS ESD"
- moved on the sheet: H10, H11, H12, H7, H8, H9, J_VIK_IN_INTC_2, J_VIK_OUT_SENS_3, J_VIK_OUT_SW_3

Commit message: Work on PCBs.
Parts:
- removed FB_USB_1: (no value), Inductor_SMD:L_0805_2012Metric, symbol Device:FerriteBead
- removed F_USB_2: SMD0805-050-16V, Fuse:Fuse_0805_2012Metric, symbol Device:Fuse
- removed J_USB_1: USB_C_Receptacle_USB2.0_16P, Connector_USB:USB_C_Receptacle_HRO_TYPE-C-31-M-12, symbol Connector:USB_C_Receptacle_USB2.0_16P
- removed R_MAT_1, R_MAT_11, R_MAT_12, R_MAT_2, R_MAT_21, R_MAT_22, R_MAT_31: 10K, Resistor_SMD:R_0201_0603Metric_Pad0.64x0.40mm_HandSolder, symbol Device:R
- removed R_MON_3: 820K, Resistor_SMD:R_0603_1608Metric, symbol Device:R
- removed R_MON_4: 2M, Resistor_SMD:R_0603_1608Metric, symbol Device:R
- removed R_USB_1, R_USB_2: 5.1K, Resistor_SMD:R_0201_0603Metric_Pad0.64x0.40mm_HandSolder, symbol Device:R
- removed SW_BAT_1: SW_SPST, library:AS11CH, symbol Switch:SW_SPST
- removed U_MAT_1: MCP23017_SS, Package_SO:SSOP-28_5.3x10.2mm_P0.65mm, symbol Interface_Expansion:MCP23017x-x-SS
- removed U_POW_1: XC6220B331MR, Package_TO_SOT_SMD:SOT-23-5, symbol Regulator_Linear:XC6220B331MR
- renumbered JP_CHG_2 to JP_CHG_1, J_VIK_IN_INTC_2 to J_VIK_IN_INTC_1, J_VIK_OUT_DISP_3 to J_VIK_OUT_DISP_2, J_VIK_OUT_SENS_3 to J_VIK_OUT_SENS_2, J_VIK_OUT_SW_3 to J_VIK_OUT_SW_2, R_CHG_3 to R_CHG_1, R_CHG_4 to R_CHG_2, U_CHG_2 to U_CHG_1
Connections:
- net BATT_MON is gone; now on net CS_DIS2: J_VIK_IN_INTC_1.8 (RGB_DO)
- net C0 is gone; now on net SDA: J_VIK_OUT_SW_2.3 (SDA)
- net C1 is gone; now on net SCL: J_VIK_OUT_SW_2.4 (SCL)
- net C3 is gone; now on net VUSB: J_VIK_OUT_SW_2.6 (5V)
- net C4 is gone; now on net D-: J_VIK_OUT_SW_2.7 (GP_AD1)
- net C5 is gone; now on net MOSI: J_VIK_OUT_SW_2.8 (MOSI)
- net R0 is gone; now on net D+: J_VIK_OUT_SW_2.9 (GP_AD2)
- net R2 is gone; now on net MISO: J_VIK_OUT_SW_2.11 (MISO)
- net R3 is gone; now on net SCLK: J_VIK_OUT_SW_2.12 (SCLK)
- net D+: now also J_VIK_IN_INTC_1.4 (GP_AD2); no longer J_VIK_IN_INTC_1.6 (GP_AD1)
- net D-: now also J_VIK_IN_INTC_1.6 (GP_AD1); no longer J_VIK_IN_INTC_1.4 (GP_AD2)
- net GND: now also J_VIK_IN_INTC_1.13 (MP), J_VIK_IN_INTC_1.14 (MP), J_VIK_OUT_DISP_2.13 (MP), J_VIK_OUT_DISP_2.14 (MP), J_VIK_OUT_SENS_2.13 (MP), J_VIK_OUT_SENS_2.14 (MP), J_VIK_OUT_SW_2.13 (MP), J_VIK_OUT_SW_2.14 (MP)
- net VBAT: now also J_BAT_1.1 (Pin_1)
- net VCC: now also J_VIK_OUT_DISP_2.6 (5V)
- net VUSB: now also U_CHG_1.4 (V_{DD})
- removed net 5V: J_VIK_OUT_DISP_2.6 (5V), U_CHG_1.4 (V_{DD})
- net C2: no longer names the net of J_VIK_OUT_SW_2.5 (RGB_DO)
- net R1: no longer names the net of J_VIK_OUT_SW_2.10 (SPI_CS)
- no-connect marks 14 -> 7
Other:
- note removed: "Battery Monitor"
- note removed: "Port"
- note removed: "VBUS ESD"

Commit message: Tentatively finish PCBs.
Parts:
- added C1, C2: 4.7uF, Capacitor_SMD:C_1206_3216Metric_Pad1.33x1.80mm_HandSolder, symbol Device:C
- J_BAT_1: symbol Connector_Generic:Conn_01x02 -> Connector_Generic_MountingPin:Conn_01x02_MountingPin
- R_CHG_1, R_CHG_2, R_POW_1: footprint Resistor_SMD:R_0201_0603Metric_Pad0.64x0.40mm_HandSolder -> Resistor_SMD:R_1206_3216Metric_Pad1.30x1.75mm_HandSolder
Connections:
- net CHG_STAT: now also J_VIK_OUT_SW_2.5 (RGB_DO)
- net GND: now also J_BAT_1.MP (MountPin), C1.2, C2.2
- net VBAT: now also C1.1
- net VUSB: now also C2.1
- no-connect marks 7 -> 6
Other:
- moved on the sheet: JP_CHG_1, R_CHG_1, R_CHG_2, U_CHG_1

Commit message: Add ESD protection to PCBs.
Parts:
- added U_ESD_D4, U_ESD_D5: CM1293A, Package_TO_SOT_SMD:SOT-23-6, symbol Power_Protection:SRV05-4
Connections:
- net CS_DIS2: now also U_ESD_D4.1 (IO1)
- net CS_PMW2: now also U_ESD_D4.3 (IO2)
- net GND: now also U_ESD_D4.2 (VN), U_ESD_D5.2 (VN)
- net MISO: now also U_ESD_D5.4 (IO3)
- net MOSI: now also U_ESD_D5.6 (IO4)
- net SCL: now also U_ESD_D4.4 (IO3)
- net SCLK: now also U_ESD_D5.3 (IO2)
- net SDA: now also U_ESD_D4.6 (IO4)
- net VDD: now also U_ESD_D4.5 (VP), U_ESD_D5.5 (VP)
- no-connect marks 6 -> 7
