File: pcb/matrix_plate/_restore_backup_2026-07-19T20-53-51-729/left.kicad_sch (KiCad schematic)
At the start: 31 parts

Commit message: Move diodes to front of matrix plates for cheaper assembly.
Parts:
- renumbered J_L_VIK_1 to J_L_VIK1, R_L_RST_1 to R_L_RST1, R_L_SCL_1 to R_L_SCL1, R_L_SDA_1 to R_L_SDA1, SW_RST_1 to SW_RST1, U_L_EXT_1 to U_L_EXT1
Changed lines of the file:
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@@
 		(dnp no)
 		(fields_autoplaced yes)
-		(property "Reference" "SW_RST_1"
+		(property "Reference" "SW_RST1"
 			(at 342.9 27.94 0)
 			(show_name no)
@@
 			(project "matrix_plate"
 				(path "/ff6e9c14-03d1-4298-be5c-ff86cb590acc/417aa41b-7daf-492f-bffc-85846200bac5"
-					(reference "SW_RST_1")
+					(reference "SW_RST1")
 					(unit 1)
 				)
@@
 		(dnp no)
 		(fields_autoplaced yes)
-		(property "Reference" "U_L_EXT_1"
+		(property "Reference" "U_L_EXT1"
 			(at 77.0733 27.94 0)
 			(show_name no)
@@
 			(project "matrix_plate"
 				(path "/ff6e9c14-03d1-4298-be5c-ff86cb590acc/417aa41b-7daf-492f-bffc-85846200bac5"
-					(reference "U_L_EXT_1")
+					(reference "U_L_EXT1")
 					(unit 1)
 				)
@@
 		(in_pos_files yes)
 		(dnp no)
-		(property "Reference" "R_L_RST_1"
+		(property "Reference" "R_L_RST1"
 			(at 55.88 52.07 90)
 			(show_name no)
@@
 			(project "matrix_plate"
 				(path "/ff6e9c14-03d1-4298-be5c-ff86cb590acc/417aa41b-7daf-492f-bffc-85846200bac5"
-					(reference "R_L_RST_1")
+					(reference "R_L_RST1")
 					(unit 1)
 				)
@@
 		(in_pos_files yes)
 		(dnp no)
-		(property "Reference" "J_L_VIK_1"
+		(property "Reference" "J_L_VIK1"
 			(at 313.182 42.926 0)
 			(show_name no)
@@
 			(project "matrix_plate"
 				(path "/ff6e9c14-03d1-4298-be5c-ff86cb590acc/417aa41b-7daf-492f-bffc-85846200bac5"
-					(reference "J_L_VIK_1")
+					(reference "J_L_VIK1")
 					(unit 1)
 				)
@@
 		(in_pos_files yes)
 		(dnp no)
-		(property "Reference" "R_L_SDA_1"
+		(property "Reference" "R_L_SDA1"
 			(at 44.45 33.02 0)
 			(show_name no)
@@
 			(project "matrix_plate"
 				(path "/ff6e9c14-03d1-4298-be5c-ff86cb590acc/417aa41b-7daf-492f-bffc-85846200bac5"
-					(reference "R_L_SDA_1")
+					(reference "R_L_SDA1")
 					(unit 1)
 				)
@@
 		(in_pos_files yes)
 		(dnp no)
-		(property "Reference" "R_L_SCL_1"
+		(property "Reference" "R_L_SCL1"
 			(at 44.45 43.18 0)
 			(show_name no)
@@
 			(project "matrix_plate"
 				(path "/ff6e9c14-03d1-4298-be5c-ff86cb590acc/417aa41b-7daf-492f-bffc-85846200bac5"
-					(reference "R_L_SCL_1")
-					(unit 1)
-				)
+					(reference "R_L_SCL1")
+					(unit 1)
+				)
