File: pcb/matrix_plate/_restore_backup_2026-07-19T20-53-51-729/right.kicad_sch (KiCad schematic)
At the start: 39 parts

Commit message: Move diodes to front of matrix plates for cheaper assembly.
Parts:
- renumbered FB_USB_1 to FB_USB1, F_USB_1 to F_USB1, J_USB_1 to J_USB1, J_R_VIK_1 to J_VIK_IN_SW_2, R_R_RST_1 to R_R_RST1, R_R_SCL_1 to R_R_SCK1, R_R_SDA_1 to R_R_SDA1, R_USB_2 to R_R_USB1, R_USB_1 to R_R_USB_1, U_R_EXT_1 to U_R_EXT1
Changed lines of the file:
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@@
 		(in_pos_files yes)
 		(dnp no)
-		(property "Reference" "J_R_VIK_1"
+		(property "Reference" "J_VIK_IN_SW_2"
 			(at 45.72 193.0399 0)
 			(show_name no)
@@
 			(project "matrix_plate"
 				(path "/ff6e9c14-03d1-4298-be5c-ff86cb590acc/4386d739-3b56-4538-90bf-5938d3c74d96"
-					(reference "J_R_VIK_1")
+					(reference "J_VIK_IN_SW_2")
 					(unit 1)
 				)
@@
 		(dnp no)
 		(fields_autoplaced yes)
-		(property "Reference" "J_USB_1"
+		(property "Reference" "J_USB1"
 			(at 293.37 25.4 0)
 			(show_name no)
@@
 			(project "matrix_plate"
 				(path "/ff6e9c14-03d1-4298-be5c-ff86cb590acc/4386d739-3b56-4538-90bf-5938d3c74d96"
-					(reference "J_USB_1")
+					(reference "J_USB1")
 					(unit 1)
 				)
@@
 		(in_pos_files yes)
 		(dnp no)
-		(property "Reference" "R_R_SCL_1"
+		(property "Reference" "R_R_SCK1"
 			(at 44.45 43.18 0)
 			(show_name no)
@@
 			(project "matrix_plate"
 				(path "/ff6e9c14-03d1-4298-be5c-ff86cb590acc/4386d739-3b56-4538-90bf-5938d3c74d96"
-					(reference "R_R_SCL_1")
+					(reference "R_R_SCK1")
 					(unit 1)
 				)
@@
 		(dnp no)
 		(fields_autoplaced yes)
-		(property "Reference" "F_USB_1"
+		(property "Reference" "F_USB1"
 			(at 336.55 109.22 90)
 			(show_name no)
@@
 			(project "matrix_plate"
 				(path "/ff6e9c14-03d1-4298-be5c-ff86cb590acc/4386d739-3b56-4538-90bf-5938d3c74d96"
-					(reference "F_USB_1")
+					(reference "F_USB1")
 					(unit 1)
 				)
@@
 		(in_pos_files yes)
 		(dnp no)
-		(property "Reference" "R_USB_2"
+		(property "Reference" "R_R_USB1"
 			(at 330.2 46.99 90)
 			(show_name no)
@@
 			(project "matrix_plate"
 				(path "/ff6e9c14-03d1-4298-be5c-ff86cb590acc/4386d739-3b56-4538-90bf-5938d3c74d96"
-					(reference "R_USB_2")
+					(reference "R_R_USB1")
 					(unit 1)
 				)
@@
 		(dnp no)
 		(fields_autoplaced yes)
-		(property "Reference" "U_R_EXT_1"
+		(property "Reference" "U_R_EXT1"
 			(at 77.0733 27.94 0)
 			(show_name no)
@@
 			(project "matrix_plate"
 				(path "/ff6e9c14-03d1-4298-be5c-ff86cb590acc/4386d739-3b56-4538-90bf-5938d3c74d96"
-					(reference "U_R_EXT_1")
+					(reference "U_R_EXT1")
 					(unit 1)
 				)
@@
 		(dnp no)
 		(fields_autoplaced yes)
-		(property "Reference" "FB_USB_1"
+		(property "Reference" "FB_USB1"
 			(at 346.075 55.8291 0)
 			(show_name no)
@@
 			(project "matrix_plate"
 				(path "/ff6e9c14-03d1-4298-be5c-ff86cb590acc/4386d739-3b56-4538-90bf-5938d3c74d96"
-					(reference "FB_USB_1")
+					(reference "FB_USB1")
 					(unit 1)
 				)
@@
 		(in_pos_files yes)
 		(dnp no)
-		(property "Reference" "R_R_SDA_1"
+		(property "Reference" "R_R_SDA1"
 			(at 44.45 33.02 0)
 			(show_name no)
@@
 			(project "matrix_plate"
 				(path "/ff6e9c14-03d1-4298-be5c-ff86cb590acc/4386d739-3b56-4538-90bf-5938d3c74d96"
-					(reference "R_R_SDA_1")
+					(reference "R_R_SDA1")
 					(unit 1)
 				)
@@
 		(in_pos_files yes)
 		(dnp no)
-		(property "Reference" "R_R_RST_1"
+		(property "Reference" "R_R_RST1"
 			(at 58.42 52.07 90)
 			(show_name no)
@@
 			(project "matrix_plate"
 				(path "/ff6e9c14-03d1-4298-be5c-ff86cb590acc/4386d739-3b56-4538-90bf-5938d3c74d96"
-					(reference "R_R_RST_1")
+					(reference "R_R_RST1")
 					(unit 1)
 				)
@@
 		(dnp no)
 		(fields_autoplaced yes)
-		(property "Reference" "R_USB_1"
+		(property "Reference" "R_R_USB_1"
 			(at 330.2 31.75 90)
 			(show_name no)
@@
 			(project "matrix_plate"
 				(path "/ff6e9c14-03d1-4298-be5c-ff86cb590acc/4386d739-3b56-4538-90bf-5938d3c74d96"
-					(reference "R_USB_1")
-					(unit 1)
-				)
+					(reference "R_R_USB_1")
+					(unit 1)
+				)
